Commit message: Change reference URDF

File: tests/api/controllers/robot_urdf/reference_robot.urdf (robot description, URDF)
Before this commit: robot UR5e, 7 links, 6 joints
Links:
- removed link forearm_link_187
- removed link shoulder_link_112
- removed link upper_arm_link_136
- removed link wrist_1_link_227
- removed link wrist_2_link_251
- removed link wrist_3_link_275
- added link forearm_link; visual box size=0.01 0.01 0.01; visual box size=0.01 0.01 0.01
- added link shoulder_link; visual box size=0.01 0.01 0.01; visual box size=0.01 0.01 0.01
- added link upper_arm_link; visual box size=0.01 0.01 0.01; visual box size=0.01 0.01 0.01
- added link wrist_1_link; visual box size=0.01 0.01 0.01; visual box size=0.01 0.01 0.01
- added link wrist_2_link; visual box size=0.01 0.01 0.01; visual box size=0.01 0.01 0.01
- added link wrist_3_link; visual box size=0.01 0.01 0.01; visual box size=0.01 0.01 0.01
Joints:
- joint elbow_joint_sensor: child forearm_link_187 -> forearm_link; parent upper_arm_link_136 -> upper_arm_link
- joint shoulder_lift_joint_sensor: child upper_arm_link_136 -> upper_arm_link; parent shoulder_link_112 -> shoulder_link
- joint shoulder_pan_joint_sensor: child shoulder_link_112 -> shoulder_link
- joint wrist_1_joint_sensor: child wrist_1_link_227 -> wrist_1_link; parent forearm_link_187 -> forearm_link
- joint wrist_2_joint_sensor: child wrist_2_link_251 -> wrist_2_link; parent wrist_1_link_227 -> wrist_1_link
- joint wrist_3_joint_sensor: child wrist_3_link_275 -> wrist_3_link; parent wrist_2_link_251 -> wrist_2_link

Commit message: Update URDF reference file

File: tests/api/controllers/robot_urdf/reference_robot.urdf (robot description, URDF)
Before this commit: robot UR5e, 7 links, 6 joints
Links:
- added link base_footprint
Joints:
- added joint base_joint: type fixed, parent base_link, child base_footprint, origin xyz=0 0 0 rpy=0 0 0, axis 0 0 0

Commit message: Update test.

File: tests/api/controllers/robot_urdf/reference_robot.urdf (robot description, URDF)
Before this commit: robot UR5e, 7 links, 6 joints
Links:
- added link track_354
Joints:
- added joint wrist_3_link_track_354_joint: type fixed, parent wrist_3_link, child track_354, origin xyz=0 0.1 0 rpy=0 0 0
- joint elbow_joint_sensor: limit (none) -> lower=-3.14159 upper=3.14159 effort=150 velocity=3.14; type continuous -> revolute
- joint shoulder_lift_joint_sensor: limit (none) -> lower=-6.28319 upper=6.28319 effort=150 velocity=3.14; type continuous -> revolute
- joint shoulder_pan_joint_sensor: limit (none) -> lower=-6.28319 upper=6.28319 effort=150 velocity=3.14; type continuous -> revolute
- joint wrist_1_joint_sensor: limit (none) -> lower=-6.28319 upper=6.28319 effort=28 velocity=6.28; type continuous -> revolute
- joint wrist_2_joint_sensor: limit (none) -> lower=-6.28319 upper=6.28319 effort=28 velocity=6.28; type continuous -> revolute
- joint wrist_3_joint_sensor: limit (none) -> lower=-6.28319 upper=6.28319 effort=28 velocity=6.28; type continuous -> revolute

Commit message: Update test.

File: tests/api/controllers/robot_urdf/reference_robot.urdf (robot description, URDF)
Before this commit: robot UR5e, 8 links, 7 joints
Links:
- link base_link: geometry collision cylinder length=0.1 radius=0.076; visual cylinder length=0.1 radius=0.076
- link forearm_link: geometry collision cylinder length=0.109 radius=0.039; collision cylinder length=0.36 radius=0.038
- link shoulder_link: geometry collision cylinder length=0.093 radius=0.059; collision cylinder length=0.135 radius=0.059
- link upper_arm_link: geometry collision cylinder length=0.133 radius=0.059; collision cylinder length=0.149 radius=0.059
- link wrist_1_link: geometry collision cylinder length=0.086 radius=0.038; collision cylinder length=0.112 radius=0.038
- link wrist_2_link: geometry collision cylinder length=0.043 radius=0.038; collision cylinder length=0.108 radius=0.04
- link wrist_3_link: geometry collision cylinder length=0.018 radius=0.032; collision cylinder length=0.048 radius=0.038

Commit message: Update URDF reference document

File: tests/api/controllers/robot_urdf/reference_robot.urdf (robot description, URDF)
Before this commit: robot UR5e, 8 links, 7 joints
Links:
- link forearm_link: geometry collision cylinder length=0.05 radius=0.058; collision cylinder length=0.1 radius=0.04

Commit message: updated reference

File: tests/api/controllers/robot_urdf/reference_robot.urdf (robot description, URDF)
Before this commit: robot UR5e, 8 links, 7 joints
Joints:
- joint shoulder_lift_joint_sensor: origin xyz=0 0.138 0 rpy=0 1.5707959999869179 0 -> xyz=0 0.138 0 rpy=0 1.570796 0
- joint wrist_1_joint_sensor: origin xyz=0 0 0.392 rpy=0 1.5707959999869179 0 -> xyz=0 0 0.392 rpy=0 1.570796 0
