Commit message: Udpate tests.

File: tests/api/controllers/robot_urdf/tiago_reference.urdf (robot description, URDF)
Before this commit: robot TIAGo++, 84 links, 83 joints
Joints:
- removed joint arm_left_1_joint_sensor
- removed joint arm_left_2_joint_sensor
- removed joint arm_left_3_joint_sensor
- removed joint arm_left_4_joint_sensor
- removed joint arm_left_5_joint_sensor
- removed joint arm_left_6_joint_sensor
- removed joint arm_left_7_joint_sensor
- removed joint arm_right_1_joint_sensor
- removed joint arm_right_2_joint_sensor
- removed joint arm_right_3_joint_sensor
- removed joint arm_right_4_joint_sensor
- removed joint arm_right_5_joint_sensor
- removed joint arm_right_6_joint_sensor
- removed joint arm_right_7_joint_sensor
- removed joint head_1_joint_sensor
- removed joint head_2_joint_sensor
- removed joint left_hand_gripper_left_finger_joint_sensor
- removed joint left_hand_gripper_right_finger_joint_sensor
- removed joint right_hand_gripper_left_finger_joint_sensor
- removed joint right_hand_gripper_right_finger_joint_sensor
- removed joint torso_lift_joint_sensor
- removed joint wheel_left_joint_sensor
- removed joint wheel_right_joint_sensor
- added joint arm_left_1_joint: type revolute, parent TIAGo left arm_61030, child TIAGo_left_arm_61045, origin xyz=0.0251 0.194 -0.171 rpy=0 0 1.5708, axis 0 0 -1, limit lower=-1.11 upper=1.5 effort=43 velocity=1.95
- added joint arm_left_2_joint: type revolute, parent TIAGo_left_arm_61045, child arm_left_2_link_61078, origin xyz=0.125 0.018 -0.031 rpy=1.5708 0 0, axis 0 -3.6732051e-06 -1, limit lower=-1.11 upper=1.5 effort=43 velocity=1.95
- added joint arm_left_3_joint: type revolute, parent arm_left_2_link_61078, child arm_left_3_link_61092, origin xyz=0.0872 0 -0.0015 rpy=1.5708569 -0.0001126458 -1.5708569, axis -6.056618e-05 -6.055936e-05 -1, limit lower=-0.72 upper=3.86 effort=26 velocity=2.35
- added joint arm_left_4_joint: type revolute, parent arm_left_3_link_61092, child arm_left_4_link_61126, origin xyz=-0.02 -0.027 -0.222 rpy=2.356193 -1.5707923 2.356193, axis 2.8276386e-06 -2.8276306e-06 1, limit lower=-0.32 upper=2.29 effort=26 velocity=2.35
- added joint arm_left_5_joint: type revolute, parent arm_left_4_link_61126, child arm_left_5_link_61160, origin xyz=-0.162 0.02 0.027 rpy=3.1415927 -1.5707927 3.1415927, axis -3.6732051e-06 0 -1, limit lower=-2.07 upper=2.07 effort=3 velocity=1.95
- added joint arm_left_6_joint: type revolute, parent arm_left_5_link_61160, child arm_left_6_link_61175, origin xyz=0 0 0.15 rpy=2.356193 -1.5707923 2.356193, axis -2.8276386e-06 2.8276306e-06 -1, limit lower=-1.39 upper=1.39 effort=6.6 velocity=1.76
- added joint arm_left_7_joint: type revolute, parent arm_left_6_link_61175, child arm_left_7_link_61190, origin xyz=0.055 0 0 rpy=1.5707991 -2.8276386e-06 1.5707991, axis 2.8276306e-06 -2.8276386e-06 -1, limit lower=-2.07 upper=2.07 effort=6.6 velocity=1.76
- added joint arm_right_1_joint: type revolute, parent TIAGo right arm_59023, child TIAGo_right_arm_59038, origin xyz=0.0251 -0.194 -0.171 rpy=0 0 1.5708, axis 0 0 1, limit lower=-1.11 upper=1.5 effort=43 velocity=1.95
- added joint arm_right_2_joint: type revolute, parent TIAGo_right_arm_59038, child arm_right_2_link_59072, origin xyz=-0.125 0.018 -0.031 rpy=1.5708 0 0, axis 0 3.6732051e-06 1, limit lower=-1.11 upper=1.5 effort=43 velocity=1.95
- added joint arm_right_3_joint: type revolute, parent arm_right_2_link_59072, child arm_right_3_link_59086, origin xyz=-0.0866 0 0 rpy=1.5707991 -2.8276386e-06 1.5707991, axis -2.8276306e-06 2.8276386e-06 1, limit lower=-0.72 upper=3.86 effort=26 velocity=2.35
- added joint arm_right_4_joint: type revolute, parent arm_right_3_link_59086, child arm_right_4_link_59120, origin xyz=0.02 -0.026 -0.223 rpy=2.356193 1.5707923 -2.356193, axis 2.8276386e-06 2.8276306e-06 -1, limit lower=-0.32 upper=2.29 effort=26 velocity=2.35
- added joint arm_right_5_joint: type revolute, parent arm_right_4_link_59120, child arm_right_5_link_59154, origin xyz=0.163 0.02 0.027 rpy=-1.5707937 -1.5707911 -1.5707937, axis 1.349254e-11 5.1946963e-06 1, limit lower=-2.07 upper=2.07 effort=3 velocity=1.95
- added joint arm_right_6_joint: type revolute, parent arm_right_5_link_59154, child arm_right_6_link_59169, origin xyz=0 0 0.15 rpy=2.356193 1.5707923 -2.356193, axis 2.8276386e-06 2.8276306e-06 -1, limit lower=-1.39 upper=1.39 effort=6.6 velocity=1.76
- added joint arm_right_7_joint: type revolute, parent arm_right_6_link_59169, child arm_right_7_link_59184, origin xyz=-0.055 0 0 rpy=-1.5707991 2.8276386e-06 1.5707991, axis 2.8276306e-06 -2.8276386e-06 1, limit lower=-2.07 upper=2.07 effort=6.6 velocity=1.76
- added joint head_1_joint: type revolute, parent torso_lift_link, child head_1_link, origin xyz=0.182 0 0 rpy=0 0 0, axis 0 0 1, limit lower=-1.24 upper=1.24 effort=5.197 velocity=3
- added joint head_2_joint: type revolute, parent head_1_link, child head_2_link, origin xyz=0.005 0 0.098 rpy=1.5708 0 0, axis 0 3.6732051e-06 1, limit lower=-0.98 upper=0.79 effort=2.77 velocity=3
- added joint left_hand_gripper_left_finger_joint: type prismatic, parent left_61205, child gripper_left_finger_link_62013, origin xyz=0 0 0 rpy=0 0 3.1415, axis 1 9.265359e-05 0, limit lower=0 upper=0.045 effort=16 velocity=0.05
- added joint left_hand_gripper_right_finger_joint: type prismatic, parent left_61205, child gripper_right_finger_link_62046, origin xyz=0 0 0 rpy=0 0 0, axis 1 0 0, limit lower=0 upper=0.045 effort=16 velocity=0.05
- added joint right_hand_gripper_left_finger_joint: type prismatic, parent right_59199, child gripper_left_finger_link_60007, origin xyz=0 0 0 rpy=0 0 3.1415, axis 1 9.265359e-05 0, limit lower=0 upper=0.045 effort=16 velocity=0.05
- added joint right_hand_gripper_right_finger_joint: type prismatic, parent right_59199, child gripper_right_finger_link_60040, origin xyz=0 0 0 rpy=0 0 0, axis 1 0 0, limit lower=0 upper=0.045 effort=16 velocity=0.05
- added joint torso_lift_joint: type prismatic, parent Torso, child torso_lift_link, origin xyz=0 0 0.6 rpy=0 0 0, axis 0 0 1, limit lower=0 upper=0.35 effort=2000 velocity=0.07
- added joint wheel_left_joint: type continuous, parent base_link, child wheel_left_link, origin xyz=0 0.202 0 rpy=1.5708 0 0, axis 0 -3.6732051e-06 -1, limit effort=10 velocity=10.1523
- added joint wheel_right_joint: type continuous, parent base_link, child wheel_right_link, origin xyz=0 -0.202 0 rpy=1.5708 0 0, axis 0 -3.6732051e-06 -1, limit effort=10 velocity=10.1523

File: tests/api/controllers/robot_urdf/ur5e_reference.urdf (robot description, URDF)
Before this commit: robot UR5e, 8 links, 7 joints
Joints:
- removed joint elbow_joint_sensor
- removed joint shoulder_lift_joint_sensor
- removed joint shoulder_pan_joint_sensor
- removed joint wrist_1_joint_sensor
- removed joint wrist_2_joint_sensor
- removed joint wrist_3_joint_sensor
- added joint elbow_joint: type revolute, parent upper_arm_link, child forearm_link, origin xyz=0 -0.131 0.425 rpy=0 0 0, axis 0 1 0, limit lower=-3.14159 upper=3.14159 effort=150 velocity=3.14
- added joint shoulder_lift_joint: type revolute, parent shoulder_link, child upper_arm_link, origin xyz=0 0.138 0 rpy=0 1.570796 0, axis 0 1 0, limit lower=-6.28319 upper=6.28319 effort=150 velocity=3.14
- added joint shoulder_pan_joint: type revolute, parent base_link, child shoulder_link, origin xyz=0 0 0.163 rpy=0 0 0, axis 0 0 1, limit lower=-6.28319 upper=6.28319 effort=150 velocity=3.14
- added joint wrist_1_joint: type revolute, parent forearm_link, child wrist_1_link, origin xyz=0 0 0.392 rpy=0 1.570796 0, axis 0 1 0, limit lower=-6.28319 upper=6.28319 effort=28 velocity=6.28
- added joint wrist_2_joint: type revolute, parent wrist_1_link, child wrist_2_link, origin xyz=0 0.127 0 rpy=0 0 0, axis 0 0 1, limit lower=-6.28319 upper=6.28319 effort=28 velocity=6.28
- added joint wrist_3_joint: type revolute, parent wrist_2_link, child wrist_3_link, origin xyz=0 0 0.1 rpy=0 0 0, axis 0 1 0, limit lower=-6.28319 upper=6.28319 effort=28 velocity=6.28
