Commit message: Update references

File: tests/api/controllers/robot_urdf/tiago_reference.urdf (robot description, URDF)
Before this commit: robot TIAGo++, 88 links, 87 joints
Links:
- removed link TIAGo left arm_43965
- removed link TIAGo right arm_42520
- removed link TIAGo_left_arm_43980
- removed link TIAGo_right_arm_42535
- removed link arm_left_2_link_44013
- removed link arm_left_3_link_44027
- removed link arm_left_4_link_44061
- removed link arm_left_5_link_44095
- removed link arm_left_6_link_44110
- removed link arm_left_7_link_44125
- removed link arm_right_2_link_42569
- removed link arm_right_3_link_42583
- removed link arm_right_4_link_42617
- removed link arm_right_5_link_42651
- removed link arm_right_6_link_42666
- removed link arm_right_7_link_42681
- removed link cap screw(1)_46807
- removed link cap screw(1)_48722
- removed link cap screw(10)_47023
- removed link cap screw(10)_48938
- removed link cap screw(11)_47047
- removed link cap screw(11)_48962
- removed link cap screw(12)_47071
- removed link cap screw(12)_48986
- removed link cap screw(13)_47095
- removed link cap screw(13)_49010
- removed link cap screw(14)_47119
- removed link cap screw(14)_49034
- removed link cap screw(15)_47143
- removed link cap screw(15)_49058
- removed link cap screw(16)_47167
- removed link cap screw(16)_49082
- removed link cap screw(17)_47191
- removed link cap screw(17)_49106
- removed link cap screw(18)_47215
- removed link cap screw(18)_49130
- removed link cap screw(19)_47239
- removed link cap screw(19)_49154
- removed link cap screw(2)_46831
- removed link cap screw(2)_48746
- removed link cap screw(3)_46855
- removed link cap screw(3)_48770
- removed link cap screw(4)_46879
- removed link cap screw(4)_48794
- removed link cap screw(5)_46903
- removed link cap screw(5)_48818
- removed link cap screw(6)_46927
- removed link cap screw(6)_48842
- removed link cap screw(7)_46951
- removed link cap screw(7)_48866
- removed link cap screw(8)_46975
- removed link cap screw(8)_48890
- removed link cap screw(9)_46999
- removed link cap screw(9)_48914
- removed link cap screw_46783
- removed link cap screw_48698
- removed link gripper_left_finger_link_47267
- removed link gripper_left_finger_link_49182
- removed link gripper_right_finger_link_47300
- removed link gripper_right_finger_link_49215
- removed link left_48654
- removed link right_46739
- removed link wrist_left_ft_tool_link_44137
- removed link wrist_right_ft_tool_link_42693
- added link TIAGo left arm; collision box size=0.042 0.094 0.094; collision cylinder length=0.016 radius=0.053
- added link TIAGo right arm; collision box size=0.042 0.094 0.094; collision cylinder length=0.016 radius=0.053
- added link TIAGo_left_arm; collision box size=0.035 0.09 0.081; collision box size=0.08 0.1044 0.048
- added link TIAGo_right_arm; collision box size=0.035 0.09 0.081; collision box size=0.08 0.1044 0.048
- added link arm_left_2_link; collision cylinder length=0.048 radius=0.052; collision cylinder length=0.057 radius=0.053
- added link arm_left_3_link; collision cylinder length=0.056 radius=0.056; collision cylinder length=0.23 radius=0.053
- added link arm_left_4_link; collision cylinder length=0.056 radius=0.054; collision cylinder length=0.191 radius=0.052
- added link arm_left_5_link; collision cylinder length=0.06 radius=0.053; collision cylinder length=0.06 radius=0.057
- added link arm_left_6_link; collision cylinder length=0.013 radius=0.0226; visual cylinder length=0.013 radius=0.0226
- added link arm_left_7_link; collision cylinder length=0.0157 radius=0.0225; visual cylinder length=0.0157 radius=0.0225
- added link arm_right_2_link; collision cylinder length=0.048 radius=0.052; collision cylinder length=0.057 radius=0.053
- added link arm_right_3_link; collision cylinder length=0.056 radius=0.056; collision cylinder length=0.23 radius=0.053
- added link arm_right_4_link; collision cylinder length=0.056 radius=0.054; collision cylinder length=0.191 radius=0.052
- added link arm_right_5_link; collision cylinder length=0.06 radius=0.053; collision cylinder length=0.06 radius=0.057
- added link arm_right_6_link; collision cylinder length=0.013 radius=0.0226; visual cylinder length=0.013 radius=0.0226
- added link arm_right_7_link; collision cylinder length=0.0157 radius=0.0225; visual cylinder length=0.0157 radius=0.0225
- added link cap screw
- added link cap screw(1)
- added link cap screw(1)_23
- added link cap screw(10)
- added link cap screw(10)_14
- added link cap screw(11)
- added link cap screw(11)_13
- added link cap screw(12)
- added link cap screw(12)_12
- added link cap screw(13)
- added link cap screw(13)_11
- added link cap screw(14)
- added link cap screw(14)_10
- added link cap screw(15)
- added link cap screw(15)_9
- added link cap screw(16)
- added link cap screw(16)_8
- added link cap screw(17)
- added link cap screw(17)_7
- added link cap screw(18)
- added link cap screw(18)_6
- added link cap screw(19)
- added link cap screw(19)_5
- added link cap screw(2)
- added link cap screw(2)_22
- added link cap screw(3)
- added link cap screw(3)_21
- added link cap screw(4)
- added link cap screw(4)_20
- added link cap screw(5)
- added link cap screw(5)_19
- added link cap screw(6)
- added link cap screw(6)_18
- added link cap screw(7)
- added link cap screw(7)_17
- added link cap screw(8)
- added link cap screw(8)_16
- added link cap screw(9)
- added link cap screw(9)_15
- added link cap screw_24
- added link gripper_left_finger_link; collision box size=0.0055 0.0295 0.018; collision box size=0.0076 0.05091 0.08982
- added link gripper_left_finger_link_4; collision box size=0.0055 0.0295 0.018; collision box size=0.0076 0.05091 0.08982
- added link gripper_right_finger_link; collision box size=0.0055 0.0295 0.018; collision box size=0.0076 0.05091 0.08982
- added link gripper_right_finger_link_3; collision box size=0.0055 0.0295 0.018; collision box size=0.0076 0.05091 0.08982
- added link left; collision box size=0.04 0.0217 0.105; collision box size=0.04 0.0217 0.105
- added link right; collision box size=0.04 0.0217 0.105; collision box size=0.04 0.0217 0.105
- added link wrist_left_ft_tool_link; collision cylinder length=0.011 radius=0.0253; visual cylinder length=0.011 radius=0.0253
- added link wrist_right_ft_tool_link; collision cylinder length=0.011 radius=0.0253; visual cylinder length=0.011 radius=0.0253
Joints:
- removed joint arm_left_7_link_44125_wrist_left_ft_tool_link_44137_joint
- removed joint arm_right_7_link_42681_wrist_right_ft_tool_link_42693_joint
- removed joint hingejoint_11955
- removed joint hingejoint_11958
- removed joint hingejoint_11990
- removed joint hingejoint_11993
- removed joint hingejoint_12025
- removed joint hingejoint_12028
- removed joint hingejoint_12060
- removed joint hingejoint_12063
- removed joint left_48654_cap screw(1)_48722_joint
- removed joint left_48654_cap screw(10)_48938_joint
- removed joint left_48654_cap screw(11)_48962_joint
- removed joint left_48654_cap screw(12)_48986_joint
- removed joint left_48654_cap screw(13)_49010_joint
- removed joint left_48654_cap screw(14)_49034_joint
- removed joint left_48654_cap screw(15)_49058_joint
- removed joint left_48654_cap screw(16)_49082_joint
- removed joint left_48654_cap screw(17)_49106_joint
- removed joint left_48654_cap screw(18)_49130_joint
- removed joint left_48654_cap screw(19)_49154_joint
- removed joint left_48654_cap screw(2)_48746_joint
- removed joint left_48654_cap screw(3)_48770_joint
- removed joint left_48654_cap screw(4)_48794_joint
- removed joint left_48654_cap screw(5)_48818_joint
- removed joint left_48654_cap screw(6)_48842_joint
- removed joint left_48654_cap screw(7)_48866_joint
- removed joint left_48654_cap screw(8)_48890_joint
- removed joint left_48654_cap screw(9)_48914_joint
- removed joint left_48654_cap screw_48698_joint
- removed joint right_46739_cap screw(1)_46807_joint
- removed joint right_46739_cap screw(10)_47023_joint
- removed joint right_46739_cap screw(11)_47047_joint
- removed joint right_46739_cap screw(12)_47071_joint
- removed joint right_46739_cap screw(13)_47095_joint
- removed joint right_46739_cap screw(14)_47119_joint
- removed joint right_46739_cap screw(15)_47143_joint
- removed joint right_46739_cap screw(16)_47167_joint
- removed joint right_46739_cap screw(17)_47191_joint
- removed joint right_46739_cap screw(18)_47215_joint
- removed joint right_46739_cap screw(19)_47239_joint
- removed joint right_46739_cap screw(2)_46831_joint
- removed joint right_46739_cap screw(3)_46855_joint
- removed joint right_46739_cap screw(4)_46879_joint
- removed joint right_46739_cap screw(5)_46903_joint
- removed joint right_46739_cap screw(6)_46927_joint
- removed joint right_46739_cap screw(7)_46951_joint
- removed joint right_46739_cap screw(8)_46975_joint
- removed joint right_46739_cap screw(9)_46999_joint
- removed joint right_46739_cap screw_46783_joint
- removed joint torso_lift_link_TIAGo left arm_43965_joint
- removed joint torso_lift_link_TIAGo right arm_42520_joint
- removed joint wrist_left_ft_tool_link_44137_left_48654_joint
- removed joint wrist_right_ft_tool_link_42693_right_46739_joint
- added joint CASTER_WHEEL_BACK_LEFT_JOINT: type continuous, parent base_link, child caster_back_left_1_link, origin xyz=-0.1735 0.102 -0.0335 rpy=0 0 0, axis 0 0 1
- added joint CASTER_WHEEL_BACK_RIGHT_JOINT: type continuous, parent base_link, child caster_back_right_1_link, origin xyz=-0.1735 -0.102 -0.0335 rpy=0 0 0, axis 0 0 1
- added joint CASTER_WHEEL_FRONT_LEFT_JOINT: type continuous, parent base_link, child caster_front_left_1_link, origin xyz=0.1695 0.102 -0.0335 rpy=0 0 0, axis 0 0 1
- added joint CASTER_WHEEL_FRONT_RIGHT_JOINT: type continuous, parent base_link, child caster_front_right_1_link, origin xyz=0.1695 -0.102 -0.0335 rpy=0 0 0, axis 0 0 1
- added joint SMALL_WHEEL_JOINT: type continuous, parent caster_back_left_1_link, child caster_back_left_2_link, origin xyz=-0.016 0 -0.04 rpy=-1.5708 0 0, axis 0 -3.6732051e-06 1
- added joint SMALL_WHEEL_JOINT_0: type continuous, parent caster_back_right_1_link, child caster_back_right_2_link, origin xyz=-0.016 0 -0.04 rpy=-1.5708 0 0, axis 0 -3.6732051e-06 1
- added joint SMALL_WHEEL_JOINT_1: type continuous, parent caster_front_left_1_link, child caster_front_left_2_link, origin xyz=-0.016 0 -0.04 rpy=-1.5708 0 0, axis 0 -3.6732051e-06 1
- added joint SMALL_WHEEL_JOINT_2: type continuous, parent caster_front_right_1_link, child caster_front_right_2_link, origin xyz=-0.016 0 -0.04 rpy=-1.5708 0 0, axis 0 -3.6732051e-06 1
- added joint arm_left_7_link_wrist_left_ft_tool_link_joint: type fixed, parent arm_left_7_link, child wrist_left_ft_tool_link, origin xyz=-1.5551969e-07 1.5552013e-07 0.067725 rpy=2.356193 -1.5707923 2.356193
- added joint arm_right_7_link_wrist_right_ft_tool_link_joint: type fixed, parent arm_right_7_link, child wrist_right_ft_tool_link, origin xyz=1.5551969e-07 -1.5552013e-07 0.067725 rpy=2.356193 -1.5707923 2.356193
- added joint left_cap screw(1)_joint: type fixed, parent left, child cap screw(1), origin xyz=0.0477 0.008 -0.043 rpy=3.1415927 -1.5707927 3.1415927
- added joint left_cap screw(10)_joint: type fixed, parent left, child cap screw(10), origin xyz=-0.0477 -0.008 -0.043 rpy=3.1415927 1.5707927 3.1415927
- added joint left_cap screw(11)_joint: type fixed, parent left, child cap screw(11), origin xyz=-0.0477 -0.008 -0.0108 rpy=3.1415927 1.5707927 3.1415927
- added joint left_cap screw(12)_joint: type fixed, parent left, child cap screw(12), origin xyz=-0.0425 0.0094 -0.0945 rpy=0 0 0
- added joint left_cap screw(13)_joint: type fixed, parent left, child cap screw(13), origin xyz=0.0426 -0.0094 -0.09448 rpy=0 0 0
- added joint left_cap screw(14)_joint: type fixed, parent left, child cap screw(14), origin xyz=0 -0.033 0.0026 rpy=3.14159 0 0
- added joint left_cap screw(15)_joint: type fixed, parent left, child cap screw(15), origin xyz=0 0.033 0.0026 rpy=3.14159 0 0
- added joint left_cap screw(16)_joint: type fixed, parent left, child cap screw(16), origin xyz=-0.0433 -0.0315 0.0026 rpy=3.14159 0 0
- added joint left_cap screw(17)_joint: type fixed, parent left, child cap screw(17), origin xyz=0.0433 0.0315 0.0026 rpy=3.14159 0 0
- added joint left_cap screw(18)_joint: type fixed, parent left, child cap screw(18), origin xyz=-0.0415 0.0029 -0.0004 rpy=3.14159 0 0
- added joint left_cap screw(19)_joint: type fixed, parent left, child cap screw(19), origin xyz=0.0415 -0.0029 -0.0004 rpy=3.14159 0 0
- added joint left_cap screw(2)_joint: type fixed, parent left, child cap screw(2), origin xyz=0.0477 0.008 -0.075 rpy=3.1415927 -1.5707927 3.1415927
- added joint left_cap screw(3)_joint: type fixed, parent left, child cap screw(3), origin xyz=0.0477 -0.008 -0.075 rpy=3.1415927 -1.5707927 3.1415927
- added joint left_cap screw(4)_joint: type fixed, parent left, child cap screw(4), origin xyz=0.0477 -0.008 -0.043 rpy=3.1415927 -1.5707927 3.1415927
- added joint left_cap screw(5)_joint: type fixed, parent left, child cap screw(5), origin xyz=0.0477 -0.008 -0.0108 rpy=3.1415927 -1.5707927 3.1415927
- added joint left_cap screw(6)_joint: type fixed, parent left, child cap screw(6), origin xyz=-0.0477 0.008 -0.0108 rpy=3.1415927 1.5707927 3.1415927
- added joint left_cap screw(7)_joint: type fixed, parent left, child cap screw(7), origin xyz=-0.0477 0.008 -0.043 rpy=3.1415927 1.5707927 3.1415927
- added joint left_cap screw(8)_joint: type fixed, parent left, child cap screw(8), origin xyz=-0.0477 0.008 -0.075 rpy=3.1415927 1.5707927 3.1415927
- added joint left_cap screw(9)_joint: type fixed, parent left, child cap screw(9), origin xyz=-0.0477 -0.008 -0.075 rpy=3.1415927 1.5707927 3.1415927
- added joint left_cap screw_joint: type fixed, parent left, child cap screw, origin xyz=0.0477 0.008 -0.0108 rpy=3.1415927 -1.5707927 3.1415927
- added joint right_cap screw(1)_23_joint: type fixed, parent right, child cap screw(1)_23, origin xyz=0.0477 0.008 -0.043 rpy=3.1415927 -1.5707927 3.1415927
- added joint right_cap screw(10)_14_joint: type fixed, parent right, child cap screw(10)_14, origin xyz=-0.0477 -0.008 -0.043 rpy=3.1415927 1.5707927 3.1415927
- added joint right_cap screw(11)_13_joint: type fixed, parent right, child cap screw(11)_13, origin xyz=-0.0477 -0.008 -0.0108 rpy=3.1415927 1.5707927 3.1415927
- added joint right_cap screw(12)_12_joint: type fixed, parent right, child cap screw(12)_12, origin xyz=-0.0425 0.0094 -0.0945 rpy=0 0 0
- added joint right_cap screw(13)_11_joint: type fixed, parent right, child cap screw(13)_11, origin xyz=0.0426 -0.0094 -0.09448 rpy=0 0 0
- added joint right_cap screw(14)_10_joint: type fixed, parent right, child cap screw(14)_10, origin xyz=0 -0.033 0.0026 rpy=3.14159 0 0
- added joint right_cap screw(15)_9_joint: type fixed, parent right, child cap screw(15)_9, origin xyz=0 0.033 0.0026 rpy=3.14159 0 0
- added joint right_cap screw(16)_8_joint: type fixed, parent right, child cap screw(16)_8, origin xyz=-0.0433 -0.0315 0.0026 rpy=3.14159 0 0
- added joint right_cap screw(17)_7_joint: type fixed, parent right, child cap screw(17)_7, origin xyz=0.0433 0.0315 0.0026 rpy=3.14159 0 0
- added joint right_cap screw(18)_6_joint: type fixed, parent right, child cap screw(18)_6, origin xyz=-0.0415 0.0029 -0.0004 rpy=3.14159 0 0
- added joint right_cap screw(19)_5_joint: type fixed, parent right, child cap screw(19)_5, origin xyz=0.0415 -0.0029 -0.0004 rpy=3.14159 0 0
- added joint right_cap screw(2)_22_joint: type fixed, parent right, child cap screw(2)_22, origin xyz=0.0477 0.008 -0.075 rpy=3.1415927 -1.5707927 3.1415927
- added joint right_cap screw(3)_21_joint: type fixed, parent right, child cap screw(3)_21, origin xyz=0.0477 -0.008 -0.075 rpy=3.1415927 -1.5707927 3.1415927
- added joint right_cap screw(4)_20_joint: type fixed, parent right, child cap screw(4)_20, origin xyz=0.0477 -0.008 -0.043 rpy=3.1415927 -1.5707927 3.1415927
- added joint right_cap screw(5)_19_joint: type fixed, parent right, child cap screw(5)_19, origin xyz=0.0477 -0.008 -0.0108 rpy=3.1415927 -1.5707927 3.1415927
- added joint right_cap screw(6)_18_joint: type fixed, parent right, child cap screw(6)_18, origin xyz=-0.0477 0.008 -0.0108 rpy=3.1415927 1.5707927 3.1415927
- added joint right_cap screw(7)_17_joint: type fixed, parent right, child cap screw(7)_17, origin xyz=-0.0477 0.008 -0.043 rpy=3.1415927 1.5707927 3.1415927
- added joint right_cap screw(8)_16_joint: type fixed, parent right, child cap screw(8)_16, origin xyz=-0.0477 0.008 -0.075 rpy=3.1415927 1.5707927 3.1415927
- added joint right_cap screw(9)_15_joint: type fixed, parent right, child cap screw(9)_15, origin xyz=-0.0477 -0.008 -0.075 rpy=3.1415927 1.5707927 3.1415927
- added joint right_cap screw_24_joint: type fixed, parent right, child cap screw_24, origin xyz=0.0477 0.008 -0.0108 rpy=3.1415927 -1.5707927 3.1415927
- added joint torso_lift_link_TIAGo left arm_joint: type fixed, parent torso_lift_link, child TIAGo left arm, origin xyz=0 0 0 rpy=0 0 0
- added joint torso_lift_link_TIAGo right arm_joint: type fixed, parent torso_lift_link, child TIAGo right arm, origin xyz=1.3492402e-12 -3.6732052e-07 0 rpy=0 0 4.6928203e-06
- added joint wrist_left_ft_tool_link_left_joint: type fixed, parent wrist_left_ft_tool_link, child left, origin xyz=0.016 -5.877128e-08 0 rpy=-2.356193 1.5707923 0.78539306
- added joint wrist_right_ft_tool_link_right_joint: type fixed, parent wrist_right_ft_tool_link, child right, origin xyz=0.016 -5.877128e-08 0 rpy=-2.356193 1.5707923 0.78539306
- joint arm_left_1_joint: child TIAGo_left_arm_43980 -> TIAGo_left_arm; parent TIAGo left arm_43965 -> TIAGo left arm
- joint arm_left_2_joint: child arm_left_2_link_44013 -> arm_left_2_link; parent TIAGo_left_arm_43980 -> TIAGo_left_arm
- joint arm_left_3_joint: child arm_left_3_link_44027 -> arm_left_3_link; parent arm_left_2_link_44013 -> arm_left_2_link
- joint arm_left_4_joint: child arm_left_4_link_44061 -> arm_left_4_link; parent arm_left_3_link_44027 -> arm_left_3_link
- joint arm_left_5_joint: child arm_left_5_link_44095 -> arm_left_5_link; parent arm_left_4_link_44061 -> arm_left_4_link
- joint arm_left_6_joint: child arm_left_6_link_44110 -> arm_left_6_link; parent arm_left_5_link_44095 -> arm_left_5_link
- joint arm_left_7_joint: child arm_left_7_link_44125 -> arm_left_7_link; parent arm_left_6_link_44110 -> arm_left_6_link
- joint arm_right_1_joint: child TIAGo_right_arm_42535 -> TIAGo_right_arm; parent TIAGo right arm_42520 -> TIAGo right arm
- joint arm_right_2_joint: child arm_right_2_link_42569 -> arm_right_2_link; parent TIAGo_right_arm_42535 -> TIAGo_right_arm
- joint arm_right_3_joint: child arm_right_3_link_42583 -> arm_right_3_link; parent arm_right_2_link_42569 -> arm_right_2_link
- joint arm_right_4_joint: child arm_right_4_link_42617 -> arm_right_4_link; parent arm_right_3_link_42583 -> arm_right_3_link
- joint arm_right_5_joint: child arm_right_5_link_42651 -> arm_right_5_link; parent arm_right_4_link_42617 -> arm_right_4_link
- joint arm_right_6_joint: child arm_right_6_link_42666 -> arm_right_6_link; parent arm_right_5_link_42651 -> arm_right_5_link
- joint arm_right_7_joint: child arm_right_7_link_42681 -> arm_right_7_link; parent arm_right_6_link_42666 -> arm_right_6_link
- joint left_hand_gripper_left_finger_joint: child gripper_left_finger_link_49182 -> gripper_left_finger_link; parent left_48654 -> left
- joint left_hand_gripper_right_finger_joint: child gripper_right_finger_link_49215 -> gripper_right_finger_link; parent left_48654 -> left
- joint right_hand_gripper_left_finger_joint: child gripper_left_finger_link_47267 -> gripper_left_finger_link_4; parent right_46739 -> right
- joint right_hand_gripper_right_finger_joint: child gripper_right_finger_link_47300 -> gripper_right_finger_link_3; parent right_46739 -> right

Commit message: revert change

File: tests/api/controllers/robot_urdf/tiago_reference.urdf (robot description, URDF)
Before this commit: robot TIAGo++, 89 links, 88 joints
Joints:
- joint base_link_Hokuyo URG-04LX-UG01_joint: origin xyz=0.202 0 -0.004 rpy=0 0 0 -> xyz=0.202 0 -0.004 rpy=1.570741 0.000118 -1.570741
