Commit message: Update test.

File: tests/api/controllers/robot_urdf/prob3_reference.urdf (robot description, URDF)
Before this commit: robot P-Rob3, 19 links, 18 joints
Links:
- removed link left finger_66100
- removed link link_base_tcp180_66015
- removed link right finger_66052
- added link left finger_50340; collision box size=0.022 0.014 0.014; collision box size=0.024 0.007 0.02
- added link link_base_tcp180_50255; collision cylinder length=0.07 radius=0.08; collision sphere radius=0.08
- added link right finger_50292; collision box size=0.022 0.014 0.014; collision box size=0.024 0.007 0.02
Joints:
- removed joint link_6_top_link_base_tcp180_66015_joint
- added joint link_6_top_link_base_tcp180_50255_joint: type fixed, parent link_6_top, child link_base_tcp180_50255, origin xyz=0 0 0.0985 rpy=0 0 0
- joint 7: child right finger_66052 -> right finger_50292; parent link_base_tcp180_66015 -> link_base_tcp180_50255
- joint 7 left: child left finger_66100 -> left finger_50340; origin xyz=0 0 0.07875 rpy=0.3430009 4.528642e-07 3.14159 -> xyz=0 0 0.058 rpy=0.3430009 4.528642e-07 3.14159; parent link_base_tcp180_66015 -> link_base_tcp180_50255
