Commit message: Update test.

File: tests/api/controllers/robot_urdf/tiago_reference.urdf (robot description, URDF)
Before this commit: robot TIAGo++, 84 links, 83 joints
Links:
- removed link TIAGo left arm_61030
- removed link TIAGo right arm_59023
- removed link TIAGo_left_arm_61045
- removed link TIAGo_right_arm_59038
- removed link arm_left_2_link_61078
- removed link arm_left_3_link_61092
- removed link arm_left_4_link_61126
- removed link arm_left_5_link_61160
- removed link arm_left_6_link_61175
- removed link arm_left_7_link_61190
- removed link arm_right_2_link_59072
- removed link arm_right_3_link_59086
- removed link arm_right_4_link_59120
- removed link arm_right_5_link_59154
- removed link arm_right_6_link_59169
- removed link arm_right_7_link_59184
- removed link cap screw(1)_59281
- removed link cap screw(1)_61287
- removed link cap screw(10)_59623
- removed link cap screw(10)_61629
- removed link cap screw(11)_59661
- removed link cap screw(11)_61667
- removed link cap screw(12)_59699
- removed link cap screw(12)_61705
- removed link cap screw(13)_59737
- removed link cap screw(13)_61743
- removed link cap screw(14)_59775
- removed link cap screw(14)_61781
- removed link cap screw(15)_59813
- removed link cap screw(15)_61819
- removed link cap screw(16)_59851
- removed link cap screw(16)_61857
- removed link cap screw(17)_59889
- removed link cap screw(17)_61895
- removed link cap screw(18)_59927
- removed link cap screw(18)_61933
- removed link cap screw(19)_59965
- removed link cap screw(19)_61971
- removed link cap screw(2)_59319
- removed link cap screw(2)_61325
- removed link cap screw(3)_59357
- removed link cap screw(3)_61363
- removed link cap screw(4)_59395
- removed link cap screw(4)_61401
- removed link cap screw(5)_59433
- removed link cap screw(5)_61439
- removed link cap screw(6)_59471
- removed link cap screw(6)_61477
- removed link cap screw(7)_59509
- removed link cap screw(7)_61515
- removed link cap screw(8)_59547
- removed link cap screw(8)_61553
- removed link cap screw(9)_59585
- removed link cap screw(9)_61591
- removed link cap screw_59243
- removed link cap screw_61249
- removed link gripper_left_finger_link_60007
- removed link gripper_left_finger_link_62013
- removed link gripper_right_finger_link_60040
- removed link gripper_right_finger_link_62046
- removed link left_61205
- removed link right_59199
- removed link wrist_left_ft_tool_link_61202
- removed link wrist_right_ft_tool_link_59196
- added link TIAGo left arm_44020; collision box size=0.042 0.094 0.094; collision cylinder length=0.016 radius=0.053
- added link TIAGo right arm_42575; collision box size=0.042 0.094 0.094; collision cylinder length=0.016 radius=0.053
- added link TIAGo_left_arm_44035; collision box size=0.035 0.09 0.081; collision box size=0.08 0.1044 0.048
- added link TIAGo_right_arm_42590; collision box size=0.035 0.09 0.081; collision box size=0.08 0.1044 0.048
- added link arm_left_2_link_44068; collision cylinder length=0.048 radius=0.052; collision cylinder length=0.057 radius=0.053
- added link arm_left_3_link_44082; collision cylinder length=0.056 radius=0.056; collision cylinder length=0.23 radius=0.053
- added link arm_left_4_link_44116; collision cylinder length=0.056 radius=0.054; collision cylinder length=0.191 radius=0.052
- added link arm_left_5_link_44150; collision cylinder length=0.06 radius=0.053; collision cylinder length=0.06 radius=0.057
- added link arm_left_6_link_44165; collision cylinder length=0.013 radius=0.0226; visual cylinder length=0.013 radius=0.0226
- added link arm_left_7_link_44180; collision cylinder length=0.0157 radius=0.0225; visual cylinder length=0.0157 radius=0.0225
- added link arm_right_2_link_42624; collision cylinder length=0.048 radius=0.052; collision cylinder length=0.057 radius=0.053
- added link arm_right_3_link_42638; collision cylinder length=0.056 radius=0.056; collision cylinder length=0.23 radius=0.053
- added link arm_right_4_link_42672; collision cylinder length=0.056 radius=0.054; collision cylinder length=0.191 radius=0.052
- added link arm_right_5_link_42706; collision cylinder length=0.06 radius=0.053; collision cylinder length=0.06 radius=0.057
- added link arm_right_6_link_42721; collision cylinder length=0.013 radius=0.0226; visual cylinder length=0.013 radius=0.0226
- added link arm_right_7_link_42736; collision cylinder length=0.0157 radius=0.0225; visual cylinder length=0.0157 radius=0.0225
- added link cap screw(1)_46862
- added link cap screw(1)_48777
- added link cap screw(10)_47078
- added link cap screw(10)_48993
- added link cap screw(11)_47102
- added link cap screw(11)_49017
- added link cap screw(12)_47126
- added link cap screw(12)_49041
- added link cap screw(13)_47150
- added link cap screw(13)_49065
- added link cap screw(14)_47174
- added link cap screw(14)_49089
- added link cap screw(15)_47198
- added link cap screw(15)_49113
- added link cap screw(16)_47222
- added link cap screw(16)_49137
- added link cap screw(17)_47246
- added link cap screw(17)_49161
- added link cap screw(18)_47270
- added link cap screw(18)_49185
- added link cap screw(19)_47294
- added link cap screw(19)_49209
- added link cap screw(2)_46886
- added link cap screw(2)_48801
- added link cap screw(3)_46910
- added link cap screw(3)_48825
- added link cap screw(4)_46934
- added link cap screw(4)_48849
- added link cap screw(5)_46958
- added link cap screw(5)_48873
- added link cap screw(6)_46982
- added link cap screw(6)_48897
- added link cap screw(7)_47006
- added link cap screw(7)_48921
- added link cap screw(8)_47030
- added link cap screw(8)_48945
- added link cap screw(9)_47054
- added link cap screw(9)_48969
- added link cap screw_46838
- added link cap screw_48753
- added link gripper_left_finger_link_47322; collision box size=0.0055 0.0295 0.018; collision box size=0.0076 0.05091 0.08982
- added link gripper_left_finger_link_49237; collision box size=0.0055 0.0295 0.018; collision box size=0.0076 0.05091 0.08982
- added link gripper_right_finger_link_47355; collision box size=0.0055 0.0295 0.018; collision box size=0.0076 0.05091 0.08982
- added link gripper_right_finger_link_49270; collision box size=0.0055 0.0295 0.018; collision box size=0.0076 0.05091 0.08982
- added link left_48709; collision box size=0.04 0.0217 0.105; collision box size=0.04 0.0217 0.105
- added link right_46794; collision box size=0.04 0.0217 0.105; collision box size=0.04 0.0217 0.105
- added link wrist_left_ft_tool_link_44192; collision cylinder length=0.011 radius=0.0253; visual cylinder length=0.011 radius=0.0253
- added link wrist_right_ft_tool_link_42748; collision cylinder length=0.011 radius=0.0253; visual cylinder length=0.011 radius=0.0253
Joints:
- removed joint arm_left_7_link_61190_wrist_left_ft_tool_link_61202_joint
- removed joint arm_right_7_link_59184_wrist_right_ft_tool_link_59196_joint
- removed joint hingejoint_16536
- removed joint hingejoint_16539
- removed joint hingejoint_16571
- removed joint hingejoint_16574
- removed joint hingejoint_16606
- removed joint hingejoint_16609
- removed joint hingejoint_16641
- removed joint hingejoint_16644
- removed joint left_61205_cap screw(1)_61287_joint
- removed joint left_61205_cap screw(10)_61629_joint
- removed joint left_61205_cap screw(11)_61667_joint
- removed joint left_61205_cap screw(12)_61705_joint
- removed joint left_61205_cap screw(13)_61743_joint
- removed joint left_61205_cap screw(14)_61781_joint
- removed joint left_61205_cap screw(15)_61819_joint
- removed joint left_61205_cap screw(16)_61857_joint
- removed joint left_61205_cap screw(17)_61895_joint
- removed joint left_61205_cap screw(18)_61933_joint
- removed joint left_61205_cap screw(19)_61971_joint
- removed joint left_61205_cap screw(2)_61325_joint
- removed joint left_61205_cap screw(3)_61363_joint
- removed joint left_61205_cap screw(4)_61401_joint
- removed joint left_61205_cap screw(5)_61439_joint
- removed joint left_61205_cap screw(6)_61477_joint
- removed joint left_61205_cap screw(7)_61515_joint
- removed joint left_61205_cap screw(8)_61553_joint
- removed joint left_61205_cap screw(9)_61591_joint
- removed joint left_61205_cap screw_61249_joint
- removed joint right_59199_cap screw(1)_59281_joint
- removed joint right_59199_cap screw(10)_59623_joint
- removed joint right_59199_cap screw(11)_59661_joint
- removed joint right_59199_cap screw(12)_59699_joint
- removed joint right_59199_cap screw(13)_59737_joint
- removed joint right_59199_cap screw(14)_59775_joint
- removed joint right_59199_cap screw(15)_59813_joint
- removed joint right_59199_cap screw(16)_59851_joint
- removed joint right_59199_cap screw(17)_59889_joint
- removed joint right_59199_cap screw(18)_59927_joint
- removed joint right_59199_cap screw(19)_59965_joint
- removed joint right_59199_cap screw(2)_59319_joint
- removed joint right_59199_cap screw(3)_59357_joint
- removed joint right_59199_cap screw(4)_59395_joint
- removed joint right_59199_cap screw(5)_59433_joint
- removed joint right_59199_cap screw(6)_59471_joint
- removed joint right_59199_cap screw(7)_59509_joint
- removed joint right_59199_cap screw(8)_59547_joint
- removed joint right_59199_cap screw(9)_59585_joint
- removed joint right_59199_cap screw_59243_joint
- removed joint torso_lift_link_TIAGo left arm_61030_joint
- removed joint torso_lift_link_TIAGo right arm_59023_joint
- removed joint wrist_left_ft_tool_link_61202_left_61205_joint
- removed joint wrist_right_ft_tool_link_59196_right_59199_joint
- added joint arm_left_7_link_44180_wrist_left_ft_tool_link_44192_joint: type fixed, parent arm_left_7_link_44180, child wrist_left_ft_tool_link_44192, origin xyz=-1.5551969e-07 1.5552013e-07 0.067725 rpy=2.356193 -1.5707923 2.356193
- added joint arm_right_7_link_42736_wrist_right_ft_tool_link_42748_joint: type fixed, parent arm_right_7_link_42736, child wrist_right_ft_tool_link_42748, origin xyz=1.5551969e-07 -1.5552013e-07 0.067725 rpy=2.356193 -1.5707923 2.356193
- added joint hingejoint_12010: type continuous, parent base_link, child caster_front_right_1_link, origin xyz=0.1695 -0.102 -0.0335 rpy=0 0 0, axis 0 0 1
- added joint hingejoint_12013: type continuous, parent caster_front_right_1_link, child caster_front_right_2_link, origin xyz=-0.016 0 -0.04 rpy=-1.5708 0 0, axis 0 -3.6732051e-06 1
- added joint hingejoint_12045: type continuous, parent base_link, child caster_front_left_1_link, origin xyz=0.1695 0.102 -0.0335 rpy=0 0 0, axis 0 0 1
- added joint hingejoint_12048: type continuous, parent caster_front_left_1_link, child caster_front_left_2_link, origin xyz=-0.016 0 -0.04 rpy=-1.5708 0 0, axis 0 -3.6732051e-06 1
- added joint hingejoint_12080: type continuous, parent base_link, child caster_back_right_1_link, origin xyz=-0.1735 -0.102 -0.0335 rpy=0 0 0, axis 0 0 1
- added joint hingejoint_12083: type continuous, parent caster_back_right_1_link, child caster_back_right_2_link, origin xyz=-0.016 0 -0.04 rpy=-1.5708 0 0, axis 0 -3.6732051e-06 1
- added joint hingejoint_12115: type continuous, parent base_link, child caster_back_left_1_link, origin xyz=-0.1735 0.102 -0.0335 rpy=0 0 0, axis 0 0 1
- added joint hingejoint_12118: type continuous, parent caster_back_left_1_link, child caster_back_left_2_link, origin xyz=-0.016 0 -0.04 rpy=-1.5708 0 0, axis 0 -3.6732051e-06 1
- added joint left_48709_cap screw(1)_48777_joint: type fixed, parent left_48709, child cap screw(1)_48777, origin xyz=0.0477 0.008 -0.043 rpy=3.1415927 -1.5707927 3.1415927
- added joint left_48709_cap screw(10)_48993_joint: type fixed, parent left_48709, child cap screw(10)_48993, origin xyz=-0.0477 -0.008 -0.043 rpy=3.1415927 1.5707927 3.1415927
- added joint left_48709_cap screw(11)_49017_joint: type fixed, parent left_48709, child cap screw(11)_49017, origin xyz=-0.0477 -0.008 -0.0108 rpy=3.1415927 1.5707927 3.1415927
- added joint left_48709_cap screw(12)_49041_joint: type fixed, parent left_48709, child cap screw(12)_49041, origin xyz=-0.0425 0.0094 -0.0945 rpy=0 0 0
- added joint left_48709_cap screw(13)_49065_joint: type fixed, parent left_48709, child cap screw(13)_49065, origin xyz=0.0426 -0.0094 -0.09448 rpy=0 0 0
- added joint left_48709_cap screw(14)_49089_joint: type fixed, parent left_48709, child cap screw(14)_49089, origin xyz=0 -0.033 0.0026 rpy=3.14159 0 0
- added joint left_48709_cap screw(15)_49113_joint: type fixed, parent left_48709, child cap screw(15)_49113, origin xyz=0 0.033 0.0026 rpy=3.14159 0 0
- added joint left_48709_cap screw(16)_49137_joint: type fixed, parent left_48709, child cap screw(16)_49137, origin xyz=-0.0433 -0.0315 0.0026 rpy=3.14159 0 0
- added joint left_48709_cap screw(17)_49161_joint: type fixed, parent left_48709, child cap screw(17)_49161, origin xyz=0.0433 0.0315 0.0026 rpy=3.14159 0 0
- added joint left_48709_cap screw(18)_49185_joint: type fixed, parent left_48709, child cap screw(18)_49185, origin xyz=-0.0415 0.0029 -0.0004 rpy=3.14159 0 0
- added joint left_48709_cap screw(19)_49209_joint: type fixed, parent left_48709, child cap screw(19)_49209, origin xyz=0.0415 -0.0029 -0.0004 rpy=3.14159 0 0
- added joint left_48709_cap screw(2)_48801_joint: type fixed, parent left_48709, child cap screw(2)_48801, origin xyz=0.0477 0.008 -0.075 rpy=3.1415927 -1.5707927 3.1415927
- added joint left_48709_cap screw(3)_48825_joint: type fixed, parent left_48709, child cap screw(3)_48825, origin xyz=0.0477 -0.008 -0.075 rpy=3.1415927 -1.5707927 3.1415927
- added joint left_48709_cap screw(4)_48849_joint: type fixed, parent left_48709, child cap screw(4)_48849, origin xyz=0.0477 -0.008 -0.043 rpy=3.1415927 -1.5707927 3.1415927
- added joint left_48709_cap screw(5)_48873_joint: type fixed, parent left_48709, child cap screw(5)_48873, origin xyz=0.0477 -0.008 -0.0108 rpy=3.1415927 -1.5707927 3.1415927
- added joint left_48709_cap screw(6)_48897_joint: type fixed, parent left_48709, child cap screw(6)_48897, origin xyz=-0.0477 0.008 -0.0108 rpy=3.1415927 1.5707927 3.1415927
- added joint left_48709_cap screw(7)_48921_joint: type fixed, parent left_48709, child cap screw(7)_48921, origin xyz=-0.0477 0.008 -0.043 rpy=3.1415927 1.5707927 3.1415927
- added joint left_48709_cap screw(8)_48945_joint: type fixed, parent left_48709, child cap screw(8)_48945, origin xyz=-0.0477 0.008 -0.075 rpy=3.1415927 1.5707927 3.1415927
- added joint left_48709_cap screw(9)_48969_joint: type fixed, parent left_48709, child cap screw(9)_48969, origin xyz=-0.0477 -0.008 -0.075 rpy=3.1415927 1.5707927 3.1415927
- added joint left_48709_cap screw_48753_joint: type fixed, parent left_48709, child cap screw_48753, origin xyz=0.0477 0.008 -0.0108 rpy=3.1415927 -1.5707927 3.1415927
- added joint right_46794_cap screw(1)_46862_joint: type fixed, parent right_46794, child cap screw(1)_46862, origin xyz=0.0477 0.008 -0.043 rpy=3.1415927 -1.5707927 3.1415927
- added joint right_46794_cap screw(10)_47078_joint: type fixed, parent right_46794, child cap screw(10)_47078, origin xyz=-0.0477 -0.008 -0.043 rpy=3.1415927 1.5707927 3.1415927
- added joint right_46794_cap screw(11)_47102_joint: type fixed, parent right_46794, child cap screw(11)_47102, origin xyz=-0.0477 -0.008 -0.0108 rpy=3.1415927 1.5707927 3.1415927
- added joint right_46794_cap screw(12)_47126_joint: type fixed, parent right_46794, child cap screw(12)_47126, origin xyz=-0.0425 0.0094 -0.0945 rpy=0 0 0
- added joint right_46794_cap screw(13)_47150_joint: type fixed, parent right_46794, child cap screw(13)_47150, origin xyz=0.0426 -0.0094 -0.09448 rpy=0 0 0
- added joint right_46794_cap screw(14)_47174_joint: type fixed, parent right_46794, child cap screw(14)_47174, origin xyz=0 -0.033 0.0026 rpy=3.14159 0 0
- added joint right_46794_cap screw(15)_47198_joint: type fixed, parent right_46794, child cap screw(15)_47198, origin xyz=0 0.033 0.0026 rpy=3.14159 0 0
- added joint right_46794_cap screw(16)_47222_joint: type fixed, parent right_46794, child cap screw(16)_47222, origin xyz=-0.0433 -0.0315 0.0026 rpy=3.14159 0 0
- added joint right_46794_cap screw(17)_47246_joint: type fixed, parent right_46794, child cap screw(17)_47246, origin xyz=0.0433 0.0315 0.0026 rpy=3.14159 0 0
- added joint right_46794_cap screw(18)_47270_joint: type fixed, parent right_46794, child cap screw(18)_47270, origin xyz=-0.0415 0.0029 -0.0004 rpy=3.14159 0 0
- added joint right_46794_cap screw(19)_47294_joint: type fixed, parent right_46794, child cap screw(19)_47294, origin xyz=0.0415 -0.0029 -0.0004 rpy=3.14159 0 0
- added joint right_46794_cap screw(2)_46886_joint: type fixed, parent right_46794, child cap screw(2)_46886, origin xyz=0.0477 0.008 -0.075 rpy=3.1415927 -1.5707927 3.1415927
- added joint right_46794_cap screw(3)_46910_joint: type fixed, parent right_46794, child cap screw(3)_46910, origin xyz=0.0477 -0.008 -0.075 rpy=3.1415927 -1.5707927 3.1415927
- added joint right_46794_cap screw(4)_46934_joint: type fixed, parent right_46794, child cap screw(4)_46934, origin xyz=0.0477 -0.008 -0.043 rpy=3.1415927 -1.5707927 3.1415927
- added joint right_46794_cap screw(5)_46958_joint: type fixed, parent right_46794, child cap screw(5)_46958, origin xyz=0.0477 -0.008 -0.0108 rpy=3.1415927 -1.5707927 3.1415927
- added joint right_46794_cap screw(6)_46982_joint: type fixed, parent right_46794, child cap screw(6)_46982, origin xyz=-0.0477 0.008 -0.0108 rpy=3.1415927 1.5707927 3.1415927
- added joint right_46794_cap screw(7)_47006_joint: type fixed, parent right_46794, child cap screw(7)_47006, origin xyz=-0.0477 0.008 -0.043 rpy=3.1415927 1.5707927 3.1415927
- added joint right_46794_cap screw(8)_47030_joint: type fixed, parent right_46794, child cap screw(8)_47030, origin xyz=-0.0477 0.008 -0.075 rpy=3.1415927 1.5707927 3.1415927
- added joint right_46794_cap screw(9)_47054_joint: type fixed, parent right_46794, child cap screw(9)_47054, origin xyz=-0.0477 -0.008 -0.075 rpy=3.1415927 1.5707927 3.1415927
- added joint right_46794_cap screw_46838_joint: type fixed, parent right_46794, child cap screw_46838, origin xyz=0.0477 0.008 -0.0108 rpy=3.1415927 -1.5707927 3.1415927
- added joint torso_lift_link_TIAGo left arm_44020_joint: type fixed, parent torso_lift_link, child TIAGo left arm_44020, origin xyz=0 0 0 rpy=0 0 0
- added joint torso_lift_link_TIAGo right arm_42575_joint: type fixed, parent torso_lift_link, child TIAGo right arm_42575, origin xyz=1.3492402e-12 -3.6732052e-07 0 rpy=0 0 4.6928203e-06
- added joint wrist_left_ft_tool_link_44192_left_48709_joint: type fixed, parent wrist_left_ft_tool_link_44192, child left_48709, origin xyz=0.016 -5.877128e-08 0 rpy=-2.356193 1.5707923 0.78539306
- added joint wrist_right_ft_tool_link_42748_right_46794_joint: type fixed, parent wrist_right_ft_tool_link_42748, child right_46794, origin xyz=0.016 -5.877128e-08 0 rpy=-2.356193 1.5707923 0.78539306
- joint arm_left_1_joint: child TIAGo_left_arm_61045 -> TIAGo_left_arm_44035; origin xyz=0.0251 0.194 -0.171 rpy=0 0 1.5708 -> xyz=0.025 0.194 -0.16 rpy=0 0 1.5708; parent TIAGo left arm_61030 -> TIAGo left arm_44020
- joint arm_left_2_joint: child arm_left_2_link_61078 -> arm_left_2_link_44068; origin xyz=0.125 0.018 -0.031 rpy=1.5708 0 0 -> xyz=0.125 0.0194 -0.042 rpy=1.5708 0 0; parent TIAGo_left_arm_61045 -> TIAGo_left_arm_44035
- joint arm_left_3_joint: child arm_left_3_link_61092 -> arm_left_3_link_44082; origin xyz=0.0872 0 -0.0015 rpy=1.5708569 -0.0001126458 -1.5708569 -> xyz=0.0895 5.5098077e-09 -1.0118208e-14 rpy=1.5708569 -0.0001126458 -1.5708569; parent arm_left_2_link_61078 -> arm_left_2_link_44068
- joint arm_left_4_joint: child arm_left_4_link_61126 -> arm_left_4_link_44116; origin xyz=-0.02 -0.027 -0.222 rpy=2.356193 -1.5707923 2.356193 -> xyz=-0.01999986 -0.026999861 -0.2197 rpy=2.356193 -1.5707923 2.356193; parent arm_left_3_link_61092 -> arm_left_3_link_44082
- joint arm_left_5_joint: child arm_left_5_link_61160 -> arm_left_5_link_44150; parent arm_left_4_link_61126 -> arm_left_4_link_44116
- joint arm_left_6_joint: child arm_left_6_link_61175 -> arm_left_6_link_44165; parent arm_left_5_link_61160 -> arm_left_5_link_44150
- joint arm_left_7_joint: child arm_left_7_link_61190 -> arm_left_7_link_44180; origin xyz=0.055 0 0 rpy=1.5707991 -2.8276386e-06 1.5707991 -> xyz=0 0 0 rpy=1.5707991 -2.8276386e-06 1.5707991; parent arm_left_6_link_61175 -> arm_left_6_link_44165
- joint arm_right_1_joint: child TIAGo_right_arm_59038 -> TIAGo_right_arm_42590; origin xyz=0.0251 -0.194 -0.171 rpy=0 0 1.5708 -> xyz=0.025 -0.194 -0.17 rpy=0 0 1.5708; parent TIAGo right arm_59023 -> TIAGo right arm_42575
- joint arm_right_2_joint: child arm_right_2_link_59072 -> arm_right_2_link_42624; origin xyz=-0.125 0.018 -0.031 rpy=1.5708 0 0 -> xyz=-0.125 0.0194 -0.032 rpy=1.5708 0 0; parent TIAGo_right_arm_59038 -> TIAGo_right_arm_42590
- joint arm_right_3_joint: child arm_right_3_link_59086 -> arm_right_3_link_42638; origin xyz=-0.0866 0 0 rpy=1.5707991 -2.8276386e-06 1.5707991 -> xyz=0.0895 5.5098077e-09 -1.0118208e-14 rpy=1.5707991 -2.8276386e-06 1.5707991; parent arm_right_2_link_59072 -> arm_right_2_link_42624
- joint arm_right_4_joint: child arm_right_4_link_59120 -> arm_right_4_link_42672; origin xyz=0.02 -0.026 -0.223 rpy=2.356193 1.5707923 -2.356193 -> xyz=0.020000502 0.0014995021 -0.3991 rpy=2.356193 1.5707923 -2.356193; parent arm_right_3_link_59086 -> arm_right_3_link_42638
- joint arm_right_5_joint: child arm_right_5_link_59154 -> arm_right_5_link_42706; origin xyz=0.163 0.02 0.027 rpy=-1.5707937 -1.5707911 -1.5707937 -> xyz=0.16300008 0.020000074 0.001 rpy=-1.5707937 -1.5707911 -1.5707937; parent arm_right_4_link_59120 -> arm_right_4_link_42672
- joint arm_right_6_joint: child arm_right_6_link_59169 -> arm_right_6_link_42721; parent arm_right_5_link_59154 -> arm_right_5_link_42706
- joint arm_right_7_joint: child arm_right_7_link_59184 -> arm_right_7_link_42736; origin xyz=-0.055 0 0 rpy=-1.5707991 2.8276386e-06 1.5707991 -> xyz=0 0 0 rpy=-1.5707991 2.8276386e-06 1.5707991; parent arm_right_6_link_59169 -> arm_right_6_link_42721
- joint base_link_base_sonar_01_link_joint: origin xyz=-0.183 -0.183 0.173 rpy=0 0 -2.3561852 -> xyz=-0.183 -0.183 0.1728 rpy=0 0 -2.3561852
- joint left_hand_gripper_left_finger_joint: child gripper_left_finger_link_62013 -> gripper_left_finger_link_49237; parent left_61205 -> left_48709
- joint left_hand_gripper_right_finger_joint: child gripper_right_finger_link_62046 -> gripper_right_finger_link_49270; parent left_61205 -> left_48709
- joint right_hand_gripper_left_finger_joint: child gripper_left_finger_link_60007 -> gripper_left_finger_link_47322; parent right_59199 -> right_46794
- joint right_hand_gripper_right_finger_joint: child gripper_right_finger_link_60040 -> gripper_right_finger_link_47355; parent right_59199 -> right_46794
- joint wheel_left_joint: origin xyz=0 0.202 0 rpy=1.5708 0 0 -> xyz=0 0.2022 0 rpy=1.5708 0 0
- joint wheel_right_joint: origin xyz=0 -0.202 0 rpy=1.5708 0 0 -> xyz=0 -0.2022 0.0002 rpy=1.5708 0 0
