Commit message: Update test.

File: tests/api/controllers/robot_urdf/ur5e_reference.urdf (robot description, URDF)
Before this commit: robot UR5e, 8 links, 7 joints
Links:
- removed link track_354
- added link track_362
Joints:
- removed joint wrist_3_link_track_354_joint
- added joint wrist_3_link_track_362_joint: type fixed, parent wrist_3_link, child track_362, origin xyz=0 0.1 0 rpy=0 0 0

Commit message: Update test.

File: tests/api/controllers/robot_urdf/prob3_reference.urdf (robot description, URDF)
Before this commit: robot P-Rob3, 19 links, 18 joints
Links:
- removed link left finger_50340
- removed link link_base_tcp180_50255
- removed link right finger_50292
- added link left finger_50332; collision box size=0.022 0.014 0.014; collision box size=0.024 0.007 0.02
- added link link_base_tcp180_50247; collision cylinder length=0.07 radius=0.08; collision sphere radius=0.08
- added link right finger_50284; collision box size=0.022 0.014 0.014; collision box size=0.024 0.007 0.02
Joints:
- removed joint link_6_top_link_base_tcp180_50255_joint
- added joint link_6_top_link_base_tcp180_50247_joint: type fixed, parent link_6_top, child link_base_tcp180_50247, origin xyz=0 0 0.0985 rpy=0 0 0
- joint 7: child right finger_50292 -> right finger_50284; parent link_base_tcp180_50255 -> link_base_tcp180_50247
- joint 7 left: child left finger_50340 -> left finger_50332; parent link_base_tcp180_50255 -> link_base_tcp180_50247

File: tests/api/controllers/robot_urdf/tiago_reference.urdf (robot description, URDF)
Before this commit: robot TIAGo++, 84 links, 83 joints
Links:
- removed link TIAGo left arm_44020
- removed link TIAGo right arm_42575
- removed link TIAGo_left_arm_44035
- removed link TIAGo_right_arm_42590
- removed link arm_left_2_link_44068
- removed link arm_left_3_link_44082
- removed link arm_left_4_link_44116
- removed link arm_left_5_link_44150
- removed link arm_left_6_link_44165
- removed link arm_left_7_link_44180
- removed link arm_right_2_link_42624
- removed link arm_right_3_link_42638
- removed link arm_right_4_link_42672
- removed link arm_right_5_link_42706
- removed link arm_right_6_link_42721
- removed link arm_right_7_link_42736
- removed link cap screw(1)_46862
- removed link cap screw(1)_48777
- removed link cap screw(10)_47078
- removed link cap screw(10)_48993
- removed link cap screw(11)_47102
- removed link cap screw(11)_49017
- removed link cap screw(12)_47126
- removed link cap screw(12)_49041
- removed link cap screw(13)_47150
- removed link cap screw(13)_49065
- removed link cap screw(14)_47174
- removed link cap screw(14)_49089
- removed link cap screw(15)_47198
- removed link cap screw(15)_49113
- removed link cap screw(16)_47222
- removed link cap screw(16)_49137
- removed link cap screw(17)_47246
- removed link cap screw(17)_49161
- removed link cap screw(18)_47270
- removed link cap screw(18)_49185
- removed link cap screw(19)_47294
- removed link cap screw(19)_49209
- removed link cap screw(2)_46886
- removed link cap screw(2)_48801
- removed link cap screw(3)_46910
- removed link cap screw(3)_48825
- removed link cap screw(4)_46934
- removed link cap screw(4)_48849
- removed link cap screw(5)_46958
- removed link cap screw(5)_48873
- removed link cap screw(6)_46982
- removed link cap screw(6)_48897
- removed link cap screw(7)_47006
- removed link cap screw(7)_48921
- removed link cap screw(8)_47030
- removed link cap screw(8)_48945
- removed link cap screw(9)_47054
- removed link cap screw(9)_48969
- removed link cap screw_46838
- removed link cap screw_48753
- removed link gripper_left_finger_link_47322
- removed link gripper_left_finger_link_49237
- removed link gripper_right_finger_link_47355
- removed link gripper_right_finger_link_49270
- removed link left_48709
- removed link right_46794
- removed link wrist_left_ft_tool_link_44192
- removed link wrist_right_ft_tool_link_42748
- added link TIAGo left arm_44012; collision box size=0.042 0.094 0.094; collision cylinder length=0.016 radius=0.053
- added link TIAGo right arm_42567; collision box size=0.042 0.094 0.094; collision cylinder length=0.016 radius=0.053
- added link TIAGo_left_arm_44027; collision box size=0.035 0.09 0.081; collision box size=0.08 0.1044 0.048
- added link TIAGo_right_arm_42582; collision box size=0.035 0.09 0.081; collision box size=0.08 0.1044 0.048
- added link arm_left_2_link_44060; collision cylinder length=0.048 radius=0.052; collision cylinder length=0.057 radius=0.053
- added link arm_left_3_link_44074; collision cylinder length=0.056 radius=0.056; collision cylinder length=0.23 radius=0.053
- added link arm_left_4_link_44108; collision cylinder length=0.056 radius=0.054; collision cylinder length=0.191 radius=0.052
- added link arm_left_5_link_44142; collision cylinder length=0.06 radius=0.053; collision cylinder length=0.06 radius=0.057
- added link arm_left_6_link_44157; collision cylinder length=0.013 radius=0.0226; visual cylinder length=0.013 radius=0.0226
- added link arm_left_7_link_44172; collision cylinder length=0.0157 radius=0.0225; visual cylinder length=0.0157 radius=0.0225
- added link arm_right_2_link_42616; collision cylinder length=0.048 radius=0.052; collision cylinder length=0.057 radius=0.053
- added link arm_right_3_link_42630; collision cylinder length=0.056 radius=0.056; collision cylinder length=0.23 radius=0.053
- added link arm_right_4_link_42664; collision cylinder length=0.056 radius=0.054; collision cylinder length=0.191 radius=0.052
- added link arm_right_5_link_42698; collision cylinder length=0.06 radius=0.053; collision cylinder length=0.06 radius=0.057
- added link arm_right_6_link_42713; collision cylinder length=0.013 radius=0.0226; visual cylinder length=0.013 radius=0.0226
- added link arm_right_7_link_42728; collision cylinder length=0.0157 radius=0.0225; visual cylinder length=0.0157 radius=0.0225
- added link cap screw(1)_46854
- added link cap screw(1)_48769
- added link cap screw(10)_47070
- added link cap screw(10)_48985
- added link cap screw(11)_47094
- added link cap screw(11)_49009
- added link cap screw(12)_47118
- added link cap screw(12)_49033
- added link cap screw(13)_47142
- added link cap screw(13)_49057
- added link cap screw(14)_47166
- added link cap screw(14)_49081
- added link cap screw(15)_47190
- added link cap screw(15)_49105
- added link cap screw(16)_47214
- added link cap screw(16)_49129
- added link cap screw(17)_47238
- added link cap screw(17)_49153
- added link cap screw(18)_47262
- added link cap screw(18)_49177
- added link cap screw(19)_47286
- added link cap screw(19)_49201
- added link cap screw(2)_46878
- added link cap screw(2)_48793
- added link cap screw(3)_46902
- added link cap screw(3)_48817
- added link cap screw(4)_46926
- added link cap screw(4)_48841
- added link cap screw(5)_46950
- added link cap screw(5)_48865
- added link cap screw(6)_46974
- added link cap screw(6)_48889
- added link cap screw(7)_46998
- added link cap screw(7)_48913
- added link cap screw(8)_47022
- added link cap screw(8)_48937
- added link cap screw(9)_47046
- added link cap screw(9)_48961
- added link cap screw_46830
- added link cap screw_48745
- added link gripper_left_finger_link_47314; collision box size=0.0055 0.0295 0.018; collision box size=0.0076 0.05091 0.08982
- added link gripper_left_finger_link_49229; collision box size=0.0055 0.0295 0.018; collision box size=0.0076 0.05091 0.08982
- added link gripper_right_finger_link_47347; collision box size=0.0055 0.0295 0.018; collision box size=0.0076 0.05091 0.08982
- added link gripper_right_finger_link_49262; collision box size=0.0055 0.0295 0.018; collision box size=0.0076 0.05091 0.08982
- added link left_48701; collision box size=0.04 0.0217 0.105; collision box size=0.04 0.0217 0.105
- added link right_46786; collision box size=0.04 0.0217 0.105; collision box size=0.04 0.0217 0.105
- added link wrist_left_ft_tool_link_44184; collision cylinder length=0.011 radius=0.0253; visual cylinder length=0.011 radius=0.0253
- added link wrist_right_ft_tool_link_42740; collision cylinder length=0.011 radius=0.0253; visual cylinder length=0.011 radius=0.0253
Joints:
- removed joint arm_left_7_link_44180_wrist_left_ft_tool_link_44192_joint
- removed joint arm_right_7_link_42736_wrist_right_ft_tool_link_42748_joint
- removed joint hingejoint_12010
- removed joint hingejoint_12013
- removed joint hingejoint_12045
- removed joint hingejoint_12048
- removed joint hingejoint_12080
- removed joint hingejoint_12083
- removed joint hingejoint_12115
- removed joint hingejoint_12118
- removed joint left_48709_cap screw(1)_48777_joint
- removed joint left_48709_cap screw(10)_48993_joint
- removed joint left_48709_cap screw(11)_49017_joint
- removed joint left_48709_cap screw(12)_49041_joint
- removed joint left_48709_cap screw(13)_49065_joint
- removed joint left_48709_cap screw(14)_49089_joint
- removed joint left_48709_cap screw(15)_49113_joint
- removed joint left_48709_cap screw(16)_49137_joint
- removed joint left_48709_cap screw(17)_49161_joint
- removed joint left_48709_cap screw(18)_49185_joint
- removed joint left_48709_cap screw(19)_49209_joint
- removed joint left_48709_cap screw(2)_48801_joint
- removed joint left_48709_cap screw(3)_48825_joint
- removed joint left_48709_cap screw(4)_48849_joint
- removed joint left_48709_cap screw(5)_48873_joint
- removed joint left_48709_cap screw(6)_48897_joint
- removed joint left_48709_cap screw(7)_48921_joint
- removed joint left_48709_cap screw(8)_48945_joint
- removed joint left_48709_cap screw(9)_48969_joint
- removed joint left_48709_cap screw_48753_joint
- removed joint right_46794_cap screw(1)_46862_joint
- removed joint right_46794_cap screw(10)_47078_joint
- removed joint right_46794_cap screw(11)_47102_joint
- removed joint right_46794_cap screw(12)_47126_joint
- removed joint right_46794_cap screw(13)_47150_joint
- removed joint right_46794_cap screw(14)_47174_joint
- removed joint right_46794_cap screw(15)_47198_joint
- removed joint right_46794_cap screw(16)_47222_joint
- removed joint right_46794_cap screw(17)_47246_joint
- removed joint right_46794_cap screw(18)_47270_joint
- removed joint right_46794_cap screw(19)_47294_joint
- removed joint right_46794_cap screw(2)_46886_joint
- removed joint right_46794_cap screw(3)_46910_joint
- removed joint right_46794_cap screw(4)_46934_joint
- removed joint right_46794_cap screw(5)_46958_joint
- removed joint right_46794_cap screw(6)_46982_joint
- removed joint right_46794_cap screw(7)_47006_joint
- removed joint right_46794_cap screw(8)_47030_joint
- removed joint right_46794_cap screw(9)_47054_joint
- removed joint right_46794_cap screw_46838_joint
- removed joint torso_lift_link_TIAGo left arm_44020_joint
- removed joint torso_lift_link_TIAGo right arm_42575_joint
- removed joint wrist_left_ft_tool_link_44192_left_48709_joint
- removed joint wrist_right_ft_tool_link_42748_right_46794_joint
- added joint arm_left_7_link_44172_wrist_left_ft_tool_link_44184_joint: type fixed, parent arm_left_7_link_44172, child wrist_left_ft_tool_link_44184, origin xyz=-1.5551969e-07 1.5552013e-07 0.067725 rpy=2.356193 -1.5707923 2.356193
- added joint arm_right_7_link_42728_wrist_right_ft_tool_link_42740_joint: type fixed, parent arm_right_7_link_42728, child wrist_right_ft_tool_link_42740, origin xyz=1.5551969e-07 -1.5552013e-07 0.067725 rpy=2.356193 -1.5707923 2.356193
- added joint hingejoint_12002: type continuous, parent base_link, child caster_front_right_1_link, origin xyz=0.1695 -0.102 -0.0335 rpy=0 0 0, axis 0 0 1
- added joint hingejoint_12005: type continuous, parent caster_front_right_1_link, child caster_front_right_2_link, origin xyz=-0.016 0 -0.04 rpy=-1.5708 0 0, axis 0 -3.6732051e-06 1
- added joint hingejoint_12037: type continuous, parent base_link, child caster_front_left_1_link, origin xyz=0.1695 0.102 -0.0335 rpy=0 0 0, axis 0 0 1
- added joint hingejoint_12040: type continuous, parent caster_front_left_1_link, child caster_front_left_2_link, origin xyz=-0.016 0 -0.04 rpy=-1.5708 0 0, axis 0 -3.6732051e-06 1
- added joint hingejoint_12072: type continuous, parent base_link, child caster_back_right_1_link, origin xyz=-0.1735 -0.102 -0.0335 rpy=0 0 0, axis 0 0 1
- added joint hingejoint_12075: type continuous, parent caster_back_right_1_link, child caster_back_right_2_link, origin xyz=-0.016 0 -0.04 rpy=-1.5708 0 0, axis 0 -3.6732051e-06 1
- added joint hingejoint_12107: type continuous, parent base_link, child caster_back_left_1_link, origin xyz=-0.1735 0.102 -0.0335 rpy=0 0 0, axis 0 0 1
- added joint hingejoint_12110: type continuous, parent caster_back_left_1_link, child caster_back_left_2_link, origin xyz=-0.016 0 -0.04 rpy=-1.5708 0 0, axis 0 -3.6732051e-06 1
- added joint left_48701_cap screw(1)_48769_joint: type fixed, parent left_48701, child cap screw(1)_48769, origin xyz=0.0477 0.008 -0.043 rpy=3.1415927 -1.5707927 3.1415927
- added joint left_48701_cap screw(10)_48985_joint: type fixed, parent left_48701, child cap screw(10)_48985, origin xyz=-0.0477 -0.008 -0.043 rpy=3.1415927 1.5707927 3.1415927
- added joint left_48701_cap screw(11)_49009_joint: type fixed, parent left_48701, child cap screw(11)_49009, origin xyz=-0.0477 -0.008 -0.0108 rpy=3.1415927 1.5707927 3.1415927
- added joint left_48701_cap screw(12)_49033_joint: type fixed, parent left_48701, child cap screw(12)_49033, origin xyz=-0.0425 0.0094 -0.0945 rpy=0 0 0
- added joint left_48701_cap screw(13)_49057_joint: type fixed, parent left_48701, child cap screw(13)_49057, origin xyz=0.0426 -0.0094 -0.09448 rpy=0 0 0
- added joint left_48701_cap screw(14)_49081_joint: type fixed, parent left_48701, child cap screw(14)_49081, origin xyz=0 -0.033 0.0026 rpy=3.14159 0 0
- added joint left_48701_cap screw(15)_49105_joint: type fixed, parent left_48701, child cap screw(15)_49105, origin xyz=0 0.033 0.0026 rpy=3.14159 0 0
- added joint left_48701_cap screw(16)_49129_joint: type fixed, parent left_48701, child cap screw(16)_49129, origin xyz=-0.0433 -0.0315 0.0026 rpy=3.14159 0 0
- added joint left_48701_cap screw(17)_49153_joint: type fixed, parent left_48701, child cap screw(17)_49153, origin xyz=0.0433 0.0315 0.0026 rpy=3.14159 0 0
- added joint left_48701_cap screw(18)_49177_joint: type fixed, parent left_48701, child cap screw(18)_49177, origin xyz=-0.0415 0.0029 -0.0004 rpy=3.14159 0 0
- added joint left_48701_cap screw(19)_49201_joint: type fixed, parent left_48701, child cap screw(19)_49201, origin xyz=0.0415 -0.0029 -0.0004 rpy=3.14159 0 0
- added joint left_48701_cap screw(2)_48793_joint: type fixed, parent left_48701, child cap screw(2)_48793, origin xyz=0.0477 0.008 -0.075 rpy=3.1415927 -1.5707927 3.1415927
- added joint left_48701_cap screw(3)_48817_joint: type fixed, parent left_48701, child cap screw(3)_48817, origin xyz=0.0477 -0.008 -0.075 rpy=3.1415927 -1.5707927 3.1415927
- added joint left_48701_cap screw(4)_48841_joint: type fixed, parent left_48701, child cap screw(4)_48841, origin xyz=0.0477 -0.008 -0.043 rpy=3.1415927 -1.5707927 3.1415927
- added joint left_48701_cap screw(5)_48865_joint: type fixed, parent left_48701, child cap screw(5)_48865, origin xyz=0.0477 -0.008 -0.0108 rpy=3.1415927 -1.5707927 3.1415927
- added joint left_48701_cap screw(6)_48889_joint: type fixed, parent left_48701, child cap screw(6)_48889, origin xyz=-0.0477 0.008 -0.0108 rpy=3.1415927 1.5707927 3.1415927
- added joint left_48701_cap screw(7)_48913_joint: type fixed, parent left_48701, child cap screw(7)_48913, origin xyz=-0.0477 0.008 -0.043 rpy=3.1415927 1.5707927 3.1415927
- added joint left_48701_cap screw(8)_48937_joint: type fixed, parent left_48701, child cap screw(8)_48937, origin xyz=-0.0477 0.008 -0.075 rpy=3.1415927 1.5707927 3.1415927
- added joint left_48701_cap screw(9)_48961_joint: type fixed, parent left_48701, child cap screw(9)_48961, origin xyz=-0.0477 -0.008 -0.075 rpy=3.1415927 1.5707927 3.1415927
- added joint left_48701_cap screw_48745_joint: type fixed, parent left_48701, child cap screw_48745, origin xyz=0.0477 0.008 -0.0108 rpy=3.1415927 -1.5707927 3.1415927
- added joint right_46786_cap screw(1)_46854_joint: type fixed, parent right_46786, child cap screw(1)_46854, origin xyz=0.0477 0.008 -0.043 rpy=3.1415927 -1.5707927 3.1415927
- added joint right_46786_cap screw(10)_47070_joint: type fixed, parent right_46786, child cap screw(10)_47070, origin xyz=-0.0477 -0.008 -0.043 rpy=3.1415927 1.5707927 3.1415927
- added joint right_46786_cap screw(11)_47094_joint: type fixed, parent right_46786, child cap screw(11)_47094, origin xyz=-0.0477 -0.008 -0.0108 rpy=3.1415927 1.5707927 3.1415927
- added joint right_46786_cap screw(12)_47118_joint: type fixed, parent right_46786, child cap screw(12)_47118, origin xyz=-0.0425 0.0094 -0.0945 rpy=0 0 0
- added joint right_46786_cap screw(13)_47142_joint: type fixed, parent right_46786, child cap screw(13)_47142, origin xyz=0.0426 -0.0094 -0.09448 rpy=0 0 0
- added joint right_46786_cap screw(14)_47166_joint: type fixed, parent right_46786, child cap screw(14)_47166, origin xyz=0 -0.033 0.0026 rpy=3.14159 0 0
- added joint right_46786_cap screw(15)_47190_joint: type fixed, parent right_46786, child cap screw(15)_47190, origin xyz=0 0.033 0.0026 rpy=3.14159 0 0
- added joint right_46786_cap screw(16)_47214_joint: type fixed, parent right_46786, child cap screw(16)_47214, origin xyz=-0.0433 -0.0315 0.0026 rpy=3.14159 0 0
- added joint right_46786_cap screw(17)_47238_joint: type fixed, parent right_46786, child cap screw(17)_47238, origin xyz=0.0433 0.0315 0.0026 rpy=3.14159 0 0
- added joint right_46786_cap screw(18)_47262_joint: type fixed, parent right_46786, child cap screw(18)_47262, origin xyz=-0.0415 0.0029 -0.0004 rpy=3.14159 0 0
- added joint right_46786_cap screw(19)_47286_joint: type fixed, parent right_46786, child cap screw(19)_47286, origin xyz=0.0415 -0.0029 -0.0004 rpy=3.14159 0 0
- added joint right_46786_cap screw(2)_46878_joint: type fixed, parent right_46786, child cap screw(2)_46878, origin xyz=0.0477 0.008 -0.075 rpy=3.1415927 -1.5707927 3.1415927
- added joint right_46786_cap screw(3)_46902_joint: type fixed, parent right_46786, child cap screw(3)_46902, origin xyz=0.0477 -0.008 -0.075 rpy=3.1415927 -1.5707927 3.1415927
- added joint right_46786_cap screw(4)_46926_joint: type fixed, parent right_46786, child cap screw(4)_46926, origin xyz=0.0477 -0.008 -0.043 rpy=3.1415927 -1.5707927 3.1415927
- added joint right_46786_cap screw(5)_46950_joint: type fixed, parent right_46786, child cap screw(5)_46950, origin xyz=0.0477 -0.008 -0.0108 rpy=3.1415927 -1.5707927 3.1415927
- added joint right_46786_cap screw(6)_46974_joint: type fixed, parent right_46786, child cap screw(6)_46974, origin xyz=-0.0477 0.008 -0.0108 rpy=3.1415927 1.5707927 3.1415927
- added joint right_46786_cap screw(7)_46998_joint: type fixed, parent right_46786, child cap screw(7)_46998, origin xyz=-0.0477 0.008 -0.043 rpy=3.1415927 1.5707927 3.1415927
- added joint right_46786_cap screw(8)_47022_joint: type fixed, parent right_46786, child cap screw(8)_47022, origin xyz=-0.0477 0.008 -0.075 rpy=3.1415927 1.5707927 3.1415927
- added joint right_46786_cap screw(9)_47046_joint: type fixed, parent right_46786, child cap screw(9)_47046, origin xyz=-0.0477 -0.008 -0.075 rpy=3.1415927 1.5707927 3.1415927
- added joint right_46786_cap screw_46830_joint: type fixed, parent right_46786, child cap screw_46830, origin xyz=0.0477 0.008 -0.0108 rpy=3.1415927 -1.5707927 3.1415927
- added joint torso_lift_link_TIAGo left arm_44012_joint: type fixed, parent torso_lift_link, child TIAGo left arm_44012, origin xyz=0 0 0 rpy=0 0 0
- added joint torso_lift_link_TIAGo right arm_42567_joint: type fixed, parent torso_lift_link, child TIAGo right arm_42567, origin xyz=1.3492402e-12 -3.6732052e-07 0 rpy=0 0 4.6928203e-06
- added joint wrist_left_ft_tool_link_44184_left_48701_joint: type fixed, parent wrist_left_ft_tool_link_44184, child left_48701, origin xyz=0.016 -5.877128e-08 0 rpy=-2.356193 1.5707923 0.78539306
- added joint wrist_right_ft_tool_link_42740_right_46786_joint: type fixed, parent wrist_right_ft_tool_link_42740, child right_46786, origin xyz=0.016 -5.877128e-08 0 rpy=-2.356193 1.5707923 0.78539306
- joint arm_left_1_joint: child TIAGo_left_arm_44035 -> TIAGo_left_arm_44027; parent TIAGo left arm_44020 -> TIAGo left arm_44012
- joint arm_left_2_joint: child arm_left_2_link_44068 -> arm_left_2_link_44060; parent TIAGo_left_arm_44035 -> TIAGo_left_arm_44027
- joint arm_left_3_joint: child arm_left_3_link_44082 -> arm_left_3_link_44074; parent arm_left_2_link_44068 -> arm_left_2_link_44060
- joint arm_left_4_joint: child arm_left_4_link_44116 -> arm_left_4_link_44108; parent arm_left_3_link_44082 -> arm_left_3_link_44074
- joint arm_left_5_joint: child arm_left_5_link_44150 -> arm_left_5_link_44142; parent arm_left_4_link_44116 -> arm_left_4_link_44108
- joint arm_left_6_joint: child arm_left_6_link_44165 -> arm_left_6_link_44157; parent arm_left_5_link_44150 -> arm_left_5_link_44142
- joint arm_left_7_joint: child arm_left_7_link_44180 -> arm_left_7_link_44172; parent arm_left_6_link_44165 -> arm_left_6_link_44157
- joint arm_right_1_joint: child TIAGo_right_arm_42590 -> TIAGo_right_arm_42582; parent TIAGo right arm_42575 -> TIAGo right arm_42567
- joint arm_right_2_joint: child arm_right_2_link_42624 -> arm_right_2_link_42616; parent TIAGo_right_arm_42590 -> TIAGo_right_arm_42582
- joint arm_right_3_joint: child arm_right_3_link_42638 -> arm_right_3_link_42630; parent arm_right_2_link_42624 -> arm_right_2_link_42616
- joint arm_right_4_joint: child arm_right_4_link_42672 -> arm_right_4_link_42664; parent arm_right_3_link_42638 -> arm_right_3_link_42630
- joint arm_right_5_joint: child arm_right_5_link_42706 -> arm_right_5_link_42698; parent arm_right_4_link_42672 -> arm_right_4_link_42664
- joint arm_right_6_joint: child arm_right_6_link_42721 -> arm_right_6_link_42713; parent arm_right_5_link_42706 -> arm_right_5_link_42698
- joint arm_right_7_joint: child arm_right_7_link_42736 -> arm_right_7_link_42728; parent arm_right_6_link_42721 -> arm_right_6_link_42713
- joint left_hand_gripper_left_finger_joint: child gripper_left_finger_link_49237 -> gripper_left_finger_link_49229; parent left_48709 -> left_48701
- joint left_hand_gripper_right_finger_joint: child gripper_right_finger_link_49270 -> gripper_right_finger_link_49262; parent left_48709 -> left_48701
- joint right_hand_gripper_left_finger_joint: child gripper_left_finger_link_47322 -> gripper_left_finger_link_47314; parent right_46794 -> right_46786
- joint right_hand_gripper_right_finger_joint: child gripper_right_finger_link_47355 -> gripper_right_finger_link_47347; parent right_46794 -> right_46786

File: tests/api/controllers/robot_urdf/ur5e_reference.urdf (robot description, URDF)
Before this commit: robot UR5e, 8 links, 7 joints
Links:
- removed link track_362
- added link track_354
Joints:
- removed joint wrist_3_link_track_362_joint
- added joint wrist_3_link_track_354_joint: type fixed, parent wrist_3_link, child track_354, origin xyz=0 0.1 0 rpy=0 0 0
