Commit message: Fixed URDF test which was broken by new UR5e model

File: tests/api/controllers/robot_urdf/prob3_reference.urdf (robot description, URDF)
Before this commit: robot P-Rob3, 19 links, 18 joints
Links:
- removed link left finger_50332
- removed link link_base_tcp180_50247
- removed link right finger_50284
- added link left finger_50293; collision box size=0.022 0.014 0.014; collision box size=0.024 0.007 0.02
- added link link_base_tcp180_50208; collision cylinder length=0.07 radius=0.08; collision sphere radius=0.08
- added link right finger_50245; collision box size=0.022 0.014 0.014; collision box size=0.024 0.007 0.02
Joints:
- removed joint link_6_top_link_base_tcp180_50247_joint
- added joint link_6_top_link_base_tcp180_50208_joint: type fixed, parent link_6_top, child link_base_tcp180_50208, origin xyz=0 0 0.0985 rpy=0 0 0
- joint 7: child right finger_50284 -> right finger_50245; parent link_base_tcp180_50247 -> link_base_tcp180_50208
- joint 7 left: child left finger_50332 -> left finger_50293; parent link_base_tcp180_50247 -> link_base_tcp180_50208

File: tests/api/controllers/robot_urdf/tiago_reference.urdf (robot description, URDF)
Before this commit: robot TIAGo++, 84 links, 83 joints
Links:
- removed link TIAGo left arm_44012
- removed link TIAGo right arm_42567
- removed link TIAGo_left_arm_44027
- removed link TIAGo_right_arm_42582
- removed link arm_left_2_link_44060
- removed link arm_left_3_link_44074
- removed link arm_left_4_link_44108
- removed link arm_left_5_link_44142
- removed link arm_left_6_link_44157
- removed link arm_left_7_link_44172
- removed link arm_right_2_link_42616
- removed link arm_right_3_link_42630
- removed link arm_right_4_link_42664
- removed link arm_right_5_link_42698
- removed link arm_right_6_link_42713
- removed link arm_right_7_link_42728
- removed link cap screw(1)_46854
- removed link cap screw(1)_48769
- removed link cap screw(10)_47070
- removed link cap screw(10)_48985
- removed link cap screw(11)_47094
- removed link cap screw(11)_49009
- removed link cap screw(12)_47118
- removed link cap screw(12)_49033
- removed link cap screw(13)_47142
- removed link cap screw(13)_49057
- removed link cap screw(14)_47166
- removed link cap screw(14)_49081
- removed link cap screw(15)_47190
- removed link cap screw(15)_49105
- removed link cap screw(16)_47214
- removed link cap screw(16)_49129
- removed link cap screw(17)_47238
- removed link cap screw(17)_49153
- removed link cap screw(18)_47262
- removed link cap screw(18)_49177
- removed link cap screw(19)_47286
- removed link cap screw(19)_49201
- removed link cap screw(2)_46878
- removed link cap screw(2)_48793
- removed link cap screw(3)_46902
- removed link cap screw(3)_48817
- removed link cap screw(4)_46926
- removed link cap screw(4)_48841
- removed link cap screw(5)_46950
- removed link cap screw(5)_48865
- removed link cap screw(6)_46974
- removed link cap screw(6)_48889
- removed link cap screw(7)_46998
- removed link cap screw(7)_48913
- removed link cap screw(8)_47022
- removed link cap screw(8)_48937
- removed link cap screw(9)_47046
- removed link cap screw(9)_48961
- removed link cap screw_46830
- removed link cap screw_48745
- removed link gripper_left_finger_link_47314
- removed link gripper_left_finger_link_49229
- removed link gripper_right_finger_link_47347
- removed link gripper_right_finger_link_49262
- removed link left_48701
- removed link right_46786
- removed link wrist_left_ft_tool_link_44184
- removed link wrist_right_ft_tool_link_42740
- added link TIAGo left arm_43973; collision box size=0.042 0.094 0.094; collision cylinder length=0.016 radius=0.053
- added link TIAGo right arm_42528; collision box size=0.042 0.094 0.094; collision cylinder length=0.016 radius=0.053
- added link TIAGo_left_arm_43988; collision box size=0.035 0.09 0.081; collision box size=0.08 0.1044 0.048
- added link TIAGo_right_arm_42543; collision box size=0.035 0.09 0.081; collision box size=0.08 0.1044 0.048
- added link arm_left_2_link_44021; collision cylinder length=0.048 radius=0.052; collision cylinder length=0.057 radius=0.053
- added link arm_left_3_link_44035; collision cylinder length=0.056 radius=0.056; collision cylinder length=0.23 radius=0.053
- added link arm_left_4_link_44069; collision cylinder length=0.056 radius=0.054; collision cylinder length=0.191 radius=0.052
- added link arm_left_5_link_44103; collision cylinder length=0.06 radius=0.053; collision cylinder length=0.06 radius=0.057
- added link arm_left_6_link_44118; collision cylinder length=0.013 radius=0.0226; visual cylinder length=0.013 radius=0.0226
- added link arm_left_7_link_44133; collision cylinder length=0.0157 radius=0.0225; visual cylinder length=0.0157 radius=0.0225
- added link arm_right_2_link_42577; collision cylinder length=0.048 radius=0.052; collision cylinder length=0.057 radius=0.053
- added link arm_right_3_link_42591; collision cylinder length=0.056 radius=0.056; collision cylinder length=0.23 radius=0.053
- added link arm_right_4_link_42625; collision cylinder length=0.056 radius=0.054; collision cylinder length=0.191 radius=0.052
- added link arm_right_5_link_42659; collision cylinder length=0.06 radius=0.053; collision cylinder length=0.06 radius=0.057
- added link arm_right_6_link_42674; collision cylinder length=0.013 radius=0.0226; visual cylinder length=0.013 radius=0.0226
- added link arm_right_7_link_42689; collision cylinder length=0.0157 radius=0.0225; visual cylinder length=0.0157 radius=0.0225
- added link cap screw(1)_46815
- added link cap screw(1)_48730
- added link cap screw(10)_47031
- added link cap screw(10)_48946
- added link cap screw(11)_47055
- added link cap screw(11)_48970
- added link cap screw(12)_47079
- added link cap screw(12)_48994
- added link cap screw(13)_47103
- added link cap screw(13)_49018
- added link cap screw(14)_47127
- added link cap screw(14)_49042
- added link cap screw(15)_47151
- added link cap screw(15)_49066
- added link cap screw(16)_47175
- added link cap screw(16)_49090
- added link cap screw(17)_47199
- added link cap screw(17)_49114
- added link cap screw(18)_47223
- added link cap screw(18)_49138
- added link cap screw(19)_47247
- added link cap screw(19)_49162
- added link cap screw(2)_46839
- added link cap screw(2)_48754
- added link cap screw(3)_46863
- added link cap screw(3)_48778
- added link cap screw(4)_46887
- added link cap screw(4)_48802
- added link cap screw(5)_46911
- added link cap screw(5)_48826
- added link cap screw(6)_46935
- added link cap screw(6)_48850
- added link cap screw(7)_46959
- added link cap screw(7)_48874
- added link cap screw(8)_46983
- added link cap screw(8)_48898
- added link cap screw(9)_47007
- added link cap screw(9)_48922
- added link cap screw_46791
- added link cap screw_48706
- added link gripper_left_finger_link_47275; collision box size=0.0055 0.0295 0.018; collision box size=0.0076 0.05091 0.08982
- added link gripper_left_finger_link_49190; collision box size=0.0055 0.0295 0.018; collision box size=0.0076 0.05091 0.08982
- added link gripper_right_finger_link_47308; collision box size=0.0055 0.0295 0.018; collision box size=0.0076 0.05091 0.08982
- added link gripper_right_finger_link_49223; collision box size=0.0055 0.0295 0.018; collision box size=0.0076 0.05091 0.08982
- added link left_48662; collision box size=0.04 0.0217 0.105; collision box size=0.04 0.0217 0.105
- added link right_46747; collision box size=0.04 0.0217 0.105; collision box size=0.04 0.0217 0.105
- added link wrist_left_ft_tool_link_44145; collision cylinder length=0.011 radius=0.0253; visual cylinder length=0.011 radius=0.0253
- added link wrist_right_ft_tool_link_42701; collision cylinder length=0.011 radius=0.0253; visual cylinder length=0.011 radius=0.0253
Joints:
- removed joint arm_left_7_link_44172_wrist_left_ft_tool_link_44184_joint
- removed joint arm_right_7_link_42728_wrist_right_ft_tool_link_42740_joint
- removed joint hingejoint_12002
- removed joint hingejoint_12005
- removed joint hingejoint_12037
- removed joint hingejoint_12040
- removed joint hingejoint_12072
- removed joint hingejoint_12075
- removed joint hingejoint_12107
- removed joint hingejoint_12110
- removed joint left_48701_cap screw(1)_48769_joint
- removed joint left_48701_cap screw(10)_48985_joint
- removed joint left_48701_cap screw(11)_49009_joint
- removed joint left_48701_cap screw(12)_49033_joint
- removed joint left_48701_cap screw(13)_49057_joint
- removed joint left_48701_cap screw(14)_49081_joint
- removed joint left_48701_cap screw(15)_49105_joint
- removed joint left_48701_cap screw(16)_49129_joint
- removed joint left_48701_cap screw(17)_49153_joint
- removed joint left_48701_cap screw(18)_49177_joint
- removed joint left_48701_cap screw(19)_49201_joint
- removed joint left_48701_cap screw(2)_48793_joint
- removed joint left_48701_cap screw(3)_48817_joint
- removed joint left_48701_cap screw(4)_48841_joint
- removed joint left_48701_cap screw(5)_48865_joint
- removed joint left_48701_cap screw(6)_48889_joint
- removed joint left_48701_cap screw(7)_48913_joint
- removed joint left_48701_cap screw(8)_48937_joint
- removed joint left_48701_cap screw(9)_48961_joint
- removed joint left_48701_cap screw_48745_joint
- removed joint right_46786_cap screw(1)_46854_joint
- removed joint right_46786_cap screw(10)_47070_joint
- removed joint right_46786_cap screw(11)_47094_joint
- removed joint right_46786_cap screw(12)_47118_joint
- removed joint right_46786_cap screw(13)_47142_joint
- removed joint right_46786_cap screw(14)_47166_joint
- removed joint right_46786_cap screw(15)_47190_joint
- removed joint right_46786_cap screw(16)_47214_joint
- removed joint right_46786_cap screw(17)_47238_joint
- removed joint right_46786_cap screw(18)_47262_joint
- removed joint right_46786_cap screw(19)_47286_joint
- removed joint right_46786_cap screw(2)_46878_joint
- removed joint right_46786_cap screw(3)_46902_joint
- removed joint right_46786_cap screw(4)_46926_joint
- removed joint right_46786_cap screw(5)_46950_joint
- removed joint right_46786_cap screw(6)_46974_joint
- removed joint right_46786_cap screw(7)_46998_joint
- removed joint right_46786_cap screw(8)_47022_joint
- removed joint right_46786_cap screw(9)_47046_joint
- removed joint right_46786_cap screw_46830_joint
- removed joint torso_lift_link_TIAGo left arm_44012_joint
- removed joint torso_lift_link_TIAGo right arm_42567_joint
- removed joint wrist_left_ft_tool_link_44184_left_48701_joint
- removed joint wrist_right_ft_tool_link_42740_right_46786_joint
- added joint arm_left_7_link_44133_wrist_left_ft_tool_link_44145_joint: type fixed, parent arm_left_7_link_44133, child wrist_left_ft_tool_link_44145, origin xyz=-1.5551969e-07 1.5552013e-07 0.067725 rpy=2.356193 -1.5707923 2.356193
- added joint arm_right_7_link_42689_wrist_right_ft_tool_link_42701_joint: type fixed, parent arm_right_7_link_42689, child wrist_right_ft_tool_link_42701, origin xyz=1.5551969e-07 -1.5552013e-07 0.067725 rpy=2.356193 -1.5707923 2.356193
- added joint hingejoint_11963: type continuous, parent base_link, child caster_front_right_1_link, origin xyz=0.1695 -0.102 -0.0335 rpy=0 0 0, axis 0 0 1
- added joint hingejoint_11966: type continuous, parent caster_front_right_1_link, child caster_front_right_2_link, origin xyz=-0.016 0 -0.04 rpy=-1.5708 0 0, axis 0 -3.6732051e-06 1
- added joint hingejoint_11998: type continuous, parent base_link, child caster_front_left_1_link, origin xyz=0.1695 0.102 -0.0335 rpy=0 0 0, axis 0 0 1
- added joint hingejoint_12001: type continuous, parent caster_front_left_1_link, child caster_front_left_2_link, origin xyz=-0.016 0 -0.04 rpy=-1.5708 0 0, axis 0 -3.6732051e-06 1
- added joint hingejoint_12033: type continuous, parent base_link, child caster_back_right_1_link, origin xyz=-0.1735 -0.102 -0.0335 rpy=0 0 0, axis 0 0 1
- added joint hingejoint_12036: type continuous, parent caster_back_right_1_link, child caster_back_right_2_link, origin xyz=-0.016 0 -0.04 rpy=-1.5708 0 0, axis 0 -3.6732051e-06 1
- added joint hingejoint_12068: type continuous, parent base_link, child caster_back_left_1_link, origin xyz=-0.1735 0.102 -0.0335 rpy=0 0 0, axis 0 0 1
- added joint hingejoint_12071: type continuous, parent caster_back_left_1_link, child caster_back_left_2_link, origin xyz=-0.016 0 -0.04 rpy=-1.5708 0 0, axis 0 -3.6732051e-06 1
- added joint left_48662_cap screw(1)_48730_joint: type fixed, parent left_48662, child cap screw(1)_48730, origin xyz=0.0477 0.008 -0.043 rpy=3.1415927 -1.5707927 3.1415927
- added joint left_48662_cap screw(10)_48946_joint: type fixed, parent left_48662, child cap screw(10)_48946, origin xyz=-0.0477 -0.008 -0.043 rpy=3.1415927 1.5707927 3.1415927
- added joint left_48662_cap screw(11)_48970_joint: type fixed, parent left_48662, child cap screw(11)_48970, origin xyz=-0.0477 -0.008 -0.0108 rpy=3.1415927 1.5707927 3.1415927
- added joint left_48662_cap screw(12)_48994_joint: type fixed, parent left_48662, child cap screw(12)_48994, origin xyz=-0.0425 0.0094 -0.0945 rpy=0 0 0
- added joint left_48662_cap screw(13)_49018_joint: type fixed, parent left_48662, child cap screw(13)_49018, origin xyz=0.0426 -0.0094 -0.09448 rpy=0 0 0
- added joint left_48662_cap screw(14)_49042_joint: type fixed, parent left_48662, child cap screw(14)_49042, origin xyz=0 -0.033 0.0026 rpy=3.14159 0 0
- added joint left_48662_cap screw(15)_49066_joint: type fixed, parent left_48662, child cap screw(15)_49066, origin xyz=0 0.033 0.0026 rpy=3.14159 0 0
- added joint left_48662_cap screw(16)_49090_joint: type fixed, parent left_48662, child cap screw(16)_49090, origin xyz=-0.0433 -0.0315 0.0026 rpy=3.14159 0 0
- added joint left_48662_cap screw(17)_49114_joint: type fixed, parent left_48662, child cap screw(17)_49114, origin xyz=0.0433 0.0315 0.0026 rpy=3.14159 0 0
- added joint left_48662_cap screw(18)_49138_joint: type fixed, parent left_48662, child cap screw(18)_49138, origin xyz=-0.0415 0.0029 -0.0004 rpy=3.14159 0 0
- added joint left_48662_cap screw(19)_49162_joint: type fixed, parent left_48662, child cap screw(19)_49162, origin xyz=0.0415 -0.0029 -0.0004 rpy=3.14159 0 0
- added joint left_48662_cap screw(2)_48754_joint: type fixed, parent left_48662, child cap screw(2)_48754, origin xyz=0.0477 0.008 -0.075 rpy=3.1415927 -1.5707927 3.1415927
- added joint left_48662_cap screw(3)_48778_joint: type fixed, parent left_48662, child cap screw(3)_48778, origin xyz=0.0477 -0.008 -0.075 rpy=3.1415927 -1.5707927 3.1415927
- added joint left_48662_cap screw(4)_48802_joint: type fixed, parent left_48662, child cap screw(4)_48802, origin xyz=0.0477 -0.008 -0.043 rpy=3.1415927 -1.5707927 3.1415927
- added joint left_48662_cap screw(5)_48826_joint: type fixed, parent left_48662, child cap screw(5)_48826, origin xyz=0.0477 -0.008 -0.0108 rpy=3.1415927 -1.5707927 3.1415927
- added joint left_48662_cap screw(6)_48850_joint: type fixed, parent left_48662, child cap screw(6)_48850, origin xyz=-0.0477 0.008 -0.0108 rpy=3.1415927 1.5707927 3.1415927
- added joint left_48662_cap screw(7)_48874_joint: type fixed, parent left_48662, child cap screw(7)_48874, origin xyz=-0.0477 0.008 -0.043 rpy=3.1415927 1.5707927 3.1415927
- added joint left_48662_cap screw(8)_48898_joint: type fixed, parent left_48662, child cap screw(8)_48898, origin xyz=-0.0477 0.008 -0.075 rpy=3.1415927 1.5707927 3.1415927
- added joint left_48662_cap screw(9)_48922_joint: type fixed, parent left_48662, child cap screw(9)_48922, origin xyz=-0.0477 -0.008 -0.075 rpy=3.1415927 1.5707927 3.1415927
- added joint left_48662_cap screw_48706_joint: type fixed, parent left_48662, child cap screw_48706, origin xyz=0.0477 0.008 -0.0108 rpy=3.1415927 -1.5707927 3.1415927
- added joint right_46747_cap screw(1)_46815_joint: type fixed, parent right_46747, child cap screw(1)_46815, origin xyz=0.0477 0.008 -0.043 rpy=3.1415927 -1.5707927 3.1415927
- added joint right_46747_cap screw(10)_47031_joint: type fixed, parent right_46747, child cap screw(10)_47031, origin xyz=-0.0477 -0.008 -0.043 rpy=3.1415927 1.5707927 3.1415927
- added joint right_46747_cap screw(11)_47055_joint: type fixed, parent right_46747, child cap screw(11)_47055, origin xyz=-0.0477 -0.008 -0.0108 rpy=3.1415927 1.5707927 3.1415927
- added joint right_46747_cap screw(12)_47079_joint: type fixed, parent right_46747, child cap screw(12)_47079, origin xyz=-0.0425 0.0094 -0.0945 rpy=0 0 0
- added joint right_46747_cap screw(13)_47103_joint: type fixed, parent right_46747, child cap screw(13)_47103, origin xyz=0.0426 -0.0094 -0.09448 rpy=0 0 0
- added joint right_46747_cap screw(14)_47127_joint: type fixed, parent right_46747, child cap screw(14)_47127, origin xyz=0 -0.033 0.0026 rpy=3.14159 0 0
- added joint right_46747_cap screw(15)_47151_joint: type fixed, parent right_46747, child cap screw(15)_47151, origin xyz=0 0.033 0.0026 rpy=3.14159 0 0
- added joint right_46747_cap screw(16)_47175_joint: type fixed, parent right_46747, child cap screw(16)_47175, origin xyz=-0.0433 -0.0315 0.0026 rpy=3.14159 0 0
- added joint right_46747_cap screw(17)_47199_joint: type fixed, parent right_46747, child cap screw(17)_47199, origin xyz=0.0433 0.0315 0.0026 rpy=3.14159 0 0
- added joint right_46747_cap screw(18)_47223_joint: type fixed, parent right_46747, child cap screw(18)_47223, origin xyz=-0.0415 0.0029 -0.0004 rpy=3.14159 0 0
- added joint right_46747_cap screw(19)_47247_joint: type fixed, parent right_46747, child cap screw(19)_47247, origin xyz=0.0415 -0.0029 -0.0004 rpy=3.14159 0 0
- added joint right_46747_cap screw(2)_46839_joint: type fixed, parent right_46747, child cap screw(2)_46839, origin xyz=0.0477 0.008 -0.075 rpy=3.1415927 -1.5707927 3.1415927
- added joint right_46747_cap screw(3)_46863_joint: type fixed, parent right_46747, child cap screw(3)_46863, origin xyz=0.0477 -0.008 -0.075 rpy=3.1415927 -1.5707927 3.1415927
- added joint right_46747_cap screw(4)_46887_joint: type fixed, parent right_46747, child cap screw(4)_46887, origin xyz=0.0477 -0.008 -0.043 rpy=3.1415927 -1.5707927 3.1415927
- added joint right_46747_cap screw(5)_46911_joint: type fixed, parent right_46747, child cap screw(5)_46911, origin xyz=0.0477 -0.008 -0.0108 rpy=3.1415927 -1.5707927 3.1415927
- added joint right_46747_cap screw(6)_46935_joint: type fixed, parent right_46747, child cap screw(6)_46935, origin xyz=-0.0477 0.008 -0.0108 rpy=3.1415927 1.5707927 3.1415927
- added joint right_46747_cap screw(7)_46959_joint: type fixed, parent right_46747, child cap screw(7)_46959, origin xyz=-0.0477 0.008 -0.043 rpy=3.1415927 1.5707927 3.1415927
- added joint right_46747_cap screw(8)_46983_joint: type fixed, parent right_46747, child cap screw(8)_46983, origin xyz=-0.0477 0.008 -0.075 rpy=3.1415927 1.5707927 3.1415927
- added joint right_46747_cap screw(9)_47007_joint: type fixed, parent right_46747, child cap screw(9)_47007, origin xyz=-0.0477 -0.008 -0.075 rpy=3.1415927 1.5707927 3.1415927
- added joint right_46747_cap screw_46791_joint: type fixed, parent right_46747, child cap screw_46791, origin xyz=0.0477 0.008 -0.0108 rpy=3.1415927 -1.5707927 3.1415927
- added joint torso_lift_link_TIAGo left arm_43973_joint: type fixed, parent torso_lift_link, child TIAGo left arm_43973, origin xyz=0 0 0 rpy=0 0 0
- added joint torso_lift_link_TIAGo right arm_42528_joint: type fixed, parent torso_lift_link, child TIAGo right arm_42528, origin xyz=1.3492402e-12 -3.6732052e-07 0 rpy=0 0 4.6928203e-06
- added joint wrist_left_ft_tool_link_44145_left_48662_joint: type fixed, parent wrist_left_ft_tool_link_44145, child left_48662, origin xyz=0.016 -5.877128e-08 0 rpy=-2.356193 1.5707923 0.78539306
- added joint wrist_right_ft_tool_link_42701_right_46747_joint: type fixed, parent wrist_right_ft_tool_link_42701, child right_46747, origin xyz=0.016 -5.877128e-08 0 rpy=-2.356193 1.5707923 0.78539306
- joint arm_left_1_joint: child TIAGo_left_arm_44027 -> TIAGo_left_arm_43988; parent TIAGo left arm_44012 -> TIAGo left arm_43973
- joint arm_left_2_joint: child arm_left_2_link_44060 -> arm_left_2_link_44021; parent TIAGo_left_arm_44027 -> TIAGo_left_arm_43988
- joint arm_left_3_joint: child arm_left_3_link_44074 -> arm_left_3_link_44035; parent arm_left_2_link_44060 -> arm_left_2_link_44021
- joint arm_left_4_joint: child arm_left_4_link_44108 -> arm_left_4_link_44069; parent arm_left_3_link_44074 -> arm_left_3_link_44035
- joint arm_left_5_joint: child arm_left_5_link_44142 -> arm_left_5_link_44103; parent arm_left_4_link_44108 -> arm_left_4_link_44069
- joint arm_left_6_joint: child arm_left_6_link_44157 -> arm_left_6_link_44118; parent arm_left_5_link_44142 -> arm_left_5_link_44103
- joint arm_left_7_joint: child arm_left_7_link_44172 -> arm_left_7_link_44133; parent arm_left_6_link_44157 -> arm_left_6_link_44118
- joint arm_right_1_joint: child TIAGo_right_arm_42582 -> TIAGo_right_arm_42543; parent TIAGo right arm_42567 -> TIAGo right arm_42528
- joint arm_right_2_joint: child arm_right_2_link_42616 -> arm_right_2_link_42577; parent TIAGo_right_arm_42582 -> TIAGo_right_arm_42543
- joint arm_right_3_joint: child arm_right_3_link_42630 -> arm_right_3_link_42591; parent arm_right_2_link_42616 -> arm_right_2_link_42577
- joint arm_right_4_joint: child arm_right_4_link_42664 -> arm_right_4_link_42625; parent arm_right_3_link_42630 -> arm_right_3_link_42591
- joint arm_right_5_joint: child arm_right_5_link_42698 -> arm_right_5_link_42659; parent arm_right_4_link_42664 -> arm_right_4_link_42625
- joint arm_right_6_joint: child arm_right_6_link_42713 -> arm_right_6_link_42674; parent arm_right_5_link_42698 -> arm_right_5_link_42659
- joint arm_right_7_joint: child arm_right_7_link_42728 -> arm_right_7_link_42689; parent arm_right_6_link_42713 -> arm_right_6_link_42674
- joint left_hand_gripper_left_finger_joint: child gripper_left_finger_link_49229 -> gripper_left_finger_link_49190; parent left_48701 -> left_48662
- joint left_hand_gripper_right_finger_joint: child gripper_right_finger_link_49262 -> gripper_right_finger_link_49223; parent left_48701 -> left_48662
- joint right_hand_gripper_left_finger_joint: child gripper_left_finger_link_47314 -> gripper_left_finger_link_47275; parent right_46786 -> right_46747
- joint right_hand_gripper_right_finger_joint: child gripper_right_finger_link_47347 -> gripper_right_finger_link_47308; parent right_46786 -> right_46747

File: tests/api/controllers/robot_urdf/ur5e_reference.urdf (robot description, URDF)
Before this commit: robot UR5e, 8 links, 7 joints
Links:
- removed link track_354
- added link track_315
Joints:
- removed joint wrist_3_link_track_354_joint
- added joint wrist_3_link_track_315_joint: type fixed, parent wrist_3_link, child track_315, origin xyz=0 0.1 0 rpy=0 0 0
