Commit message: Fixed URDF test which was broken by new UR5e model (#2715)
* Fixed URDF test which was broken by new UR5e model

* Fixed groundtruth

File: tests/api/controllers/robot_urdf/prob3_reference.urdf (robot description, URDF)
Before this commit: robot P-Rob3, 19 links, 18 joints
Links:
- removed link left finger_50332
- removed link link_base_tcp180_50247
- removed link right finger_50284
- added link left finger_50285; collision box size=0.022 0.014 0.014; collision box size=0.024 0.007 0.02
- added link link_base_tcp180_50200; collision cylinder length=0.07 radius=0.08; collision sphere radius=0.08
- added link right finger_50237; collision box size=0.022 0.014 0.014; collision box size=0.024 0.007 0.02
Joints:
- removed joint link_6_top_link_base_tcp180_50247_joint
- added joint link_6_top_link_base_tcp180_50200_joint: type fixed, parent link_6_top, child link_base_tcp180_50200, origin xyz=0 0 0.0985 rpy=0 0 0
- joint 7: child right finger_50284 -> right finger_50237; parent link_base_tcp180_50247 -> link_base_tcp180_50200
- joint 7 left: child left finger_50332 -> left finger_50285; parent link_base_tcp180_50247 -> link_base_tcp180_50200

File: tests/api/controllers/robot_urdf/tiago_reference.urdf (robot description, URDF)
Before this commit: robot TIAGo++, 84 links, 83 joints
Links:
- removed link TIAGo left arm_44012
- removed link TIAGo right arm_42567
- removed link TIAGo_left_arm_44027
- removed link TIAGo_right_arm_42582
- removed link arm_left_2_link_44060
- removed link arm_left_3_link_44074
- removed link arm_left_4_link_44108
- removed link arm_left_5_link_44142
- removed link arm_left_6_link_44157
- removed link arm_left_7_link_44172
- removed link arm_right_2_link_42616
- removed link arm_right_3_link_42630
- removed link arm_right_4_link_42664
- removed link arm_right_5_link_42698
- removed link arm_right_6_link_42713
- removed link arm_right_7_link_42728
- removed link cap screw(1)_46854
- removed link cap screw(1)_48769
- removed link cap screw(10)_47070
- removed link cap screw(10)_48985
- removed link cap screw(11)_47094
- removed link cap screw(11)_49009
- removed link cap screw(12)_47118
- removed link cap screw(12)_49033
- removed link cap screw(13)_47142
- removed link cap screw(13)_49057
- removed link cap screw(14)_47166
- removed link cap screw(14)_49081
- removed link cap screw(15)_47190
- removed link cap screw(15)_49105
- removed link cap screw(16)_47214
- removed link cap screw(16)_49129
- removed link cap screw(17)_47238
- removed link cap screw(17)_49153
- removed link cap screw(18)_47262
- removed link cap screw(18)_49177
- removed link cap screw(19)_47286
- removed link cap screw(19)_49201
- removed link cap screw(2)_46878
- removed link cap screw(2)_48793
- removed link cap screw(3)_46902
- removed link cap screw(3)_48817
- removed link cap screw(4)_46926
- removed link cap screw(4)_48841
- removed link cap screw(5)_46950
- removed link cap screw(5)_48865
- removed link cap screw(6)_46974
- removed link cap screw(6)_48889
- removed link cap screw(7)_46998
- removed link cap screw(7)_48913
- removed link cap screw(8)_47022
- removed link cap screw(8)_48937
- removed link cap screw(9)_47046
- removed link cap screw(9)_48961
- removed link cap screw_46830
- removed link cap screw_48745
- removed link gripper_left_finger_link_47314
- removed link gripper_left_finger_link_49229
- removed link gripper_right_finger_link_47347
- removed link gripper_right_finger_link_49262
- removed link left_48701
- removed link right_46786
- removed link wrist_left_ft_tool_link_44184
- removed link wrist_right_ft_tool_link_42740
- added link TIAGo left arm_43965; collision box size=0.042 0.094 0.094; collision cylinder length=0.016 radius=0.053
- added link TIAGo right arm_42520; collision box size=0.042 0.094 0.094; collision cylinder length=0.016 radius=0.053
- added link TIAGo_left_arm_43980; collision box size=0.035 0.09 0.081; collision box size=0.08 0.1044 0.048
- added link TIAGo_right_arm_42535; collision box size=0.035 0.09 0.081; collision box size=0.08 0.1044 0.048
- added link arm_left_2_link_44013; collision cylinder length=0.048 radius=0.052; collision cylinder length=0.057 radius=0.053
- added link arm_left_3_link_44027; collision cylinder length=0.056 radius=0.056; collision cylinder length=0.23 radius=0.053
- added link arm_left_4_link_44061; collision cylinder length=0.056 radius=0.054; collision cylinder length=0.191 radius=0.052
- added link arm_left_5_link_44095; collision cylinder length=0.06 radius=0.053; collision cylinder length=0.06 radius=0.057
- added link arm_left_6_link_44110; collision cylinder length=0.013 radius=0.0226; visual cylinder length=0.013 radius=0.0226
- added link arm_left_7_link_44125; collision cylinder length=0.0157 radius=0.0225; visual cylinder length=0.0157 radius=0.0225
- added link arm_right_2_link_42569; collision cylinder length=0.048 radius=0.052; collision cylinder length=0.057 radius=0.053
- added link arm_right_3_link_42583; collision cylinder length=0.056 radius=0.056; collision cylinder length=0.23 radius=0.053
- added link arm_right_4_link_42617; collision cylinder length=0.056 radius=0.054; collision cylinder length=0.191 radius=0.052
- added link arm_right_5_link_42651; collision cylinder length=0.06 radius=0.053; collision cylinder length=0.06 radius=0.057
- added link arm_right_6_link_42666; collision cylinder length=0.013 radius=0.0226; visual cylinder length=0.013 radius=0.0226
- added link arm_right_7_link_42681; collision cylinder length=0.0157 radius=0.0225; visual cylinder length=0.0157 radius=0.0225
- added link cap screw(1)_46807
- added link cap screw(1)_48722
- added link cap screw(10)_47023
- added link cap screw(10)_48938
- added link cap screw(11)_47047
- added link cap screw(11)_48962
- added link cap screw(12)_47071
- added link cap screw(12)_48986
- added link cap screw(13)_47095
- added link cap screw(13)_49010
- added link cap screw(14)_47119
- added link cap screw(14)_49034
- added link cap screw(15)_47143
- added link cap screw(15)_49058
- added link cap screw(16)_47167
- added link cap screw(16)_49082
- added link cap screw(17)_47191
- added link cap screw(17)_49106
- added link cap screw(18)_47215
- added link cap screw(18)_49130
- added link cap screw(19)_47239
- added link cap screw(19)_49154
- added link cap screw(2)_46831
- added link cap screw(2)_48746
- added link cap screw(3)_46855
- added link cap screw(3)_48770
- added link cap screw(4)_46879
- added link cap screw(4)_48794
- added link cap screw(5)_46903
- added link cap screw(5)_48818
- added link cap screw(6)_46927
- added link cap screw(6)_48842
- added link cap screw(7)_46951
- added link cap screw(7)_48866
- added link cap screw(8)_46975
- added link cap screw(8)_48890
- added link cap screw(9)_46999
- added link cap screw(9)_48914
- added link cap screw_46783
- added link cap screw_48698
- added link gripper_left_finger_link_47267; collision box size=0.0055 0.0295 0.018; collision box size=0.0076 0.05091 0.08982
- added link gripper_left_finger_link_49182; collision box size=0.0055 0.0295 0.018; collision box size=0.0076 0.05091 0.08982
- added link gripper_right_finger_link_47300; collision box size=0.0055 0.0295 0.018; collision box size=0.0076 0.05091 0.08982
- added link gripper_right_finger_link_49215; collision box size=0.0055 0.0295 0.018; collision box size=0.0076 0.05091 0.08982
- added link left_48654; collision box size=0.04 0.0217 0.105; collision box size=0.04 0.0217 0.105
- added link right_46739; collision box size=0.04 0.0217 0.105; collision box size=0.04 0.0217 0.105
- added link wrist_left_ft_tool_link_44137; collision cylinder length=0.011 radius=0.0253; visual cylinder length=0.011 radius=0.0253
- added link wrist_right_ft_tool_link_42693; collision cylinder length=0.011 radius=0.0253; visual cylinder length=0.011 radius=0.0253
Joints:
- removed joint arm_left_7_link_44172_wrist_left_ft_tool_link_44184_joint
- removed joint arm_right_7_link_42728_wrist_right_ft_tool_link_42740_joint
- removed joint hingejoint_12002
- removed joint hingejoint_12005
- removed joint hingejoint_12037
- removed joint hingejoint_12040
- removed joint hingejoint_12072
- removed joint hingejoint_12075
- removed joint hingejoint_12107
- removed joint hingejoint_12110
- removed joint left_48701_cap screw(1)_48769_joint
- removed joint left_48701_cap screw(10)_48985_joint
- removed joint left_48701_cap screw(11)_49009_joint
- removed joint left_48701_cap screw(12)_49033_joint
- removed joint left_48701_cap screw(13)_49057_joint
- removed joint left_48701_cap screw(14)_49081_joint
- removed joint left_48701_cap screw(15)_49105_joint
- removed joint left_48701_cap screw(16)_49129_joint
- removed joint left_48701_cap screw(17)_49153_joint
- removed joint left_48701_cap screw(18)_49177_joint
- removed joint left_48701_cap screw(19)_49201_joint
- removed joint left_48701_cap screw(2)_48793_joint
- removed joint left_48701_cap screw(3)_48817_joint
- removed joint left_48701_cap screw(4)_48841_joint
- removed joint left_48701_cap screw(5)_48865_joint
- removed joint left_48701_cap screw(6)_48889_joint
- removed joint left_48701_cap screw(7)_48913_joint
- removed joint left_48701_cap screw(8)_48937_joint
- removed joint left_48701_cap screw(9)_48961_joint
- removed joint left_48701_cap screw_48745_joint
- removed joint right_46786_cap screw(1)_46854_joint
- removed joint right_46786_cap screw(10)_47070_joint
- removed joint right_46786_cap screw(11)_47094_joint
- removed joint right_46786_cap screw(12)_47118_joint
- removed joint right_46786_cap screw(13)_47142_joint
- removed joint right_46786_cap screw(14)_47166_joint
- removed joint right_46786_cap screw(15)_47190_joint
- removed joint right_46786_cap screw(16)_47214_joint
- removed joint right_46786_cap screw(17)_47238_joint
- removed joint right_46786_cap screw(18)_47262_joint
- removed joint right_46786_cap screw(19)_47286_joint
- removed joint right_46786_cap screw(2)_46878_joint
- removed joint right_46786_cap screw(3)_46902_joint
- removed joint right_46786_cap screw(4)_46926_joint
- removed joint right_46786_cap screw(5)_46950_joint
- removed joint right_46786_cap screw(6)_46974_joint
- removed joint right_46786_cap screw(7)_46998_joint
- removed joint right_46786_cap screw(8)_47022_joint
- removed joint right_46786_cap screw(9)_47046_joint
- removed joint right_46786_cap screw_46830_joint
- removed joint torso_lift_link_TIAGo left arm_44012_joint
- removed joint torso_lift_link_TIAGo right arm_42567_joint
- removed joint wrist_left_ft_tool_link_44184_left_48701_joint
- removed joint wrist_right_ft_tool_link_42740_right_46786_joint
- added joint arm_left_7_link_44125_wrist_left_ft_tool_link_44137_joint: type fixed, parent arm_left_7_link_44125, child wrist_left_ft_tool_link_44137, origin xyz=-1.5551969e-07 1.5552013e-07 0.067725 rpy=2.356193 -1.5707923 2.356193
- added joint arm_right_7_link_42681_wrist_right_ft_tool_link_42693_joint: type fixed, parent arm_right_7_link_42681, child wrist_right_ft_tool_link_42693, origin xyz=1.5551969e-07 -1.5552013e-07 0.067725 rpy=2.356193 -1.5707923 2.356193
- added joint hingejoint_11955: type continuous, parent base_link, child caster_front_right_1_link, origin xyz=0.1695 -0.102 -0.0335 rpy=0 0 0, axis 0 0 1
- added joint hingejoint_11958: type continuous, parent caster_front_right_1_link, child caster_front_right_2_link, origin xyz=-0.016 0 -0.04 rpy=-1.5708 0 0, axis 0 -3.6732051e-06 1
- added joint hingejoint_11990: type continuous, parent base_link, child caster_front_left_1_link, origin xyz=0.1695 0.102 -0.0335 rpy=0 0 0, axis 0 0 1
- added joint hingejoint_11993: type continuous, parent caster_front_left_1_link, child caster_front_left_2_link, origin xyz=-0.016 0 -0.04 rpy=-1.5708 0 0, axis 0 -3.6732051e-06 1
- added joint hingejoint_12025: type continuous, parent base_link, child caster_back_right_1_link, origin xyz=-0.1735 -0.102 -0.0335 rpy=0 0 0, axis 0 0 1
- added joint hingejoint_12028: type continuous, parent caster_back_right_1_link, child caster_back_right_2_link, origin xyz=-0.016 0 -0.04 rpy=-1.5708 0 0, axis 0 -3.6732051e-06 1
- added joint hingejoint_12060: type continuous, parent base_link, child caster_back_left_1_link, origin xyz=-0.1735 0.102 -0.0335 rpy=0 0 0, axis 0 0 1
- added joint hingejoint_12063: type continuous, parent caster_back_left_1_link, child caster_back_left_2_link, origin xyz=-0.016 0 -0.04 rpy=-1.5708 0 0, axis 0 -3.6732051e-06 1
- added joint left_48654_cap screw(1)_48722_joint: type fixed, parent left_48654, child cap screw(1)_48722, origin xyz=0.0477 0.008 -0.043 rpy=3.1415927 -1.5707927 3.1415927
- added joint left_48654_cap screw(10)_48938_joint: type fixed, parent left_48654, child cap screw(10)_48938, origin xyz=-0.0477 -0.008 -0.043 rpy=3.1415927 1.5707927 3.1415927
- added joint left_48654_cap screw(11)_48962_joint: type fixed, parent left_48654, child cap screw(11)_48962, origin xyz=-0.0477 -0.008 -0.0108 rpy=3.1415927 1.5707927 3.1415927
- added joint left_48654_cap screw(12)_48986_joint: type fixed, parent left_48654, child cap screw(12)_48986, origin xyz=-0.0425 0.0094 -0.0945 rpy=0 0 0
- added joint left_48654_cap screw(13)_49010_joint: type fixed, parent left_48654, child cap screw(13)_49010, origin xyz=0.0426 -0.0094 -0.09448 rpy=0 0 0
- added joint left_48654_cap screw(14)_49034_joint: type fixed, parent left_48654, child cap screw(14)_49034, origin xyz=0 -0.033 0.0026 rpy=3.14159 0 0
- added joint left_48654_cap screw(15)_49058_joint: type fixed, parent left_48654, child cap screw(15)_49058, origin xyz=0 0.033 0.0026 rpy=3.14159 0 0
- added joint left_48654_cap screw(16)_49082_joint: type fixed, parent left_48654, child cap screw(16)_49082, origin xyz=-0.0433 -0.0315 0.0026 rpy=3.14159 0 0
- added joint left_48654_cap screw(17)_49106_joint: type fixed, parent left_48654, child cap screw(17)_49106, origin xyz=0.0433 0.0315 0.0026 rpy=3.14159 0 0
- added joint left_48654_cap screw(18)_49130_joint: type fixed, parent left_48654, child cap screw(18)_49130, origin xyz=-0.0415 0.0029 -0.0004 rpy=3.14159 0 0
- added joint left_48654_cap screw(19)_49154_joint: type fixed, parent left_48654, child cap screw(19)_49154, origin xyz=0.0415 -0.0029 -0.0004 rpy=3.14159 0 0
- added joint left_48654_cap screw(2)_48746_joint: type fixed, parent left_48654, child cap screw(2)_48746, origin xyz=0.0477 0.008 -0.075 rpy=3.1415927 -1.5707927 3.1415927
- added joint left_48654_cap screw(3)_48770_joint: type fixed, parent left_48654, child cap screw(3)_48770, origin xyz=0.0477 -0.008 -0.075 rpy=3.1415927 -1.5707927 3.1415927
- added joint left_48654_cap screw(4)_48794_joint: type fixed, parent left_48654, child cap screw(4)_48794, origin xyz=0.0477 -0.008 -0.043 rpy=3.1415927 -1.5707927 3.1415927
- added joint left_48654_cap screw(5)_48818_joint: type fixed, parent left_48654, child cap screw(5)_48818, origin xyz=0.0477 -0.008 -0.0108 rpy=3.1415927 -1.5707927 3.1415927
- added joint left_48654_cap screw(6)_48842_joint: type fixed, parent left_48654, child cap screw(6)_48842, origin xyz=-0.0477 0.008 -0.0108 rpy=3.1415927 1.5707927 3.1415927
- added joint left_48654_cap screw(7)_48866_joint: type fixed, parent left_48654, child cap screw(7)_48866, origin xyz=-0.0477 0.008 -0.043 rpy=3.1415927 1.5707927 3.1415927
- added joint left_48654_cap screw(8)_48890_joint: type fixed, parent left_48654, child cap screw(8)_48890, origin xyz=-0.0477 0.008 -0.075 rpy=3.1415927 1.5707927 3.1415927
- added joint left_48654_cap screw(9)_48914_joint: type fixed, parent left_48654, child cap screw(9)_48914, origin xyz=-0.0477 -0.008 -0.075 rpy=3.1415927 1.5707927 3.1415927
- added joint left_48654_cap screw_48698_joint: type fixed, parent left_48654, child cap screw_48698, origin xyz=0.0477 0.008 -0.0108 rpy=3.1415927 -1.5707927 3.1415927
- added joint right_46739_cap screw(1)_46807_joint: type fixed, parent right_46739, child cap screw(1)_46807, origin xyz=0.0477 0.008 -0.043 rpy=3.1415927 -1.5707927 3.1415927
- added joint right_46739_cap screw(10)_47023_joint: type fixed, parent right_46739, child cap screw(10)_47023, origin xyz=-0.0477 -0.008 -0.043 rpy=3.1415927 1.5707927 3.1415927
- added joint right_46739_cap screw(11)_47047_joint: type fixed, parent right_46739, child cap screw(11)_47047, origin xyz=-0.0477 -0.008 -0.0108 rpy=3.1415927 1.5707927 3.1415927
- added joint right_46739_cap screw(12)_47071_joint: type fixed, parent right_46739, child cap screw(12)_47071, origin xyz=-0.0425 0.0094 -0.0945 rpy=0 0 0
- added joint right_46739_cap screw(13)_47095_joint: type fixed, parent right_46739, child cap screw(13)_47095, origin xyz=0.0426 -0.0094 -0.09448 rpy=0 0 0
- added joint right_46739_cap screw(14)_47119_joint: type fixed, parent right_46739, child cap screw(14)_47119, origin xyz=0 -0.033 0.0026 rpy=3.14159 0 0
- added joint right_46739_cap screw(15)_47143_joint: type fixed, parent right_46739, child cap screw(15)_47143, origin xyz=0 0.033 0.0026 rpy=3.14159 0 0
- added joint right_46739_cap screw(16)_47167_joint: type fixed, parent right_46739, child cap screw(16)_47167, origin xyz=-0.0433 -0.0315 0.0026 rpy=3.14159 0 0
- added joint right_46739_cap screw(17)_47191_joint: type fixed, parent right_46739, child cap screw(17)_47191, origin xyz=0.0433 0.0315 0.0026 rpy=3.14159 0 0
- added joint right_46739_cap screw(18)_47215_joint: type fixed, parent right_46739, child cap screw(18)_47215, origin xyz=-0.0415 0.0029 -0.0004 rpy=3.14159 0 0
- added joint right_46739_cap screw(19)_47239_joint: type fixed, parent right_46739, child cap screw(19)_47239, origin xyz=0.0415 -0.0029 -0.0004 rpy=3.14159 0 0
- added joint right_46739_cap screw(2)_46831_joint: type fixed, parent right_46739, child cap screw(2)_46831, origin xyz=0.0477 0.008 -0.075 rpy=3.1415927 -1.5707927 3.1415927
- added joint right_46739_cap screw(3)_46855_joint: type fixed, parent right_46739, child cap screw(3)_46855, origin xyz=0.0477 -0.008 -0.075 rpy=3.1415927 -1.5707927 3.1415927
- added joint right_46739_cap screw(4)_46879_joint: type fixed, parent right_46739, child cap screw(4)_46879, origin xyz=0.0477 -0.008 -0.043 rpy=3.1415927 -1.5707927 3.1415927
- added joint right_46739_cap screw(5)_46903_joint: type fixed, parent right_46739, child cap screw(5)_46903, origin xyz=0.0477 -0.008 -0.0108 rpy=3.1415927 -1.5707927 3.1415927
- added joint right_46739_cap screw(6)_46927_joint: type fixed, parent right_46739, child cap screw(6)_46927, origin xyz=-0.0477 0.008 -0.0108 rpy=3.1415927 1.5707927 3.1415927
- added joint right_46739_cap screw(7)_46951_joint: type fixed, parent right_46739, child cap screw(7)_46951, origin xyz=-0.0477 0.008 -0.043 rpy=3.1415927 1.5707927 3.1415927
- added joint right_46739_cap screw(8)_46975_joint: type fixed, parent right_46739, child cap screw(8)_46975, origin xyz=-0.0477 0.008 -0.075 rpy=3.1415927 1.5707927 3.1415927
- added joint right_46739_cap screw(9)_46999_joint: type fixed, parent right_46739, child cap screw(9)_46999, origin xyz=-0.0477 -0.008 -0.075 rpy=3.1415927 1.5707927 3.1415927
- added joint right_46739_cap screw_46783_joint: type fixed, parent right_46739, child cap screw_46783, origin xyz=0.0477 0.008 -0.0108 rpy=3.1415927 -1.5707927 3.1415927
- added joint torso_lift_link_TIAGo left arm_43965_joint: type fixed, parent torso_lift_link, child TIAGo left arm_43965, origin xyz=0 0 0 rpy=0 0 0
- added joint torso_lift_link_TIAGo right arm_42520_joint: type fixed, parent torso_lift_link, child TIAGo right arm_42520, origin xyz=1.3492402e-12 -3.6732052e-07 0 rpy=0 0 4.6928203e-06
- added joint wrist_left_ft_tool_link_44137_left_48654_joint: type fixed, parent wrist_left_ft_tool_link_44137, child left_48654, origin xyz=0.016 -5.877128e-08 0 rpy=-2.356193 1.5707923 0.78539306
- added joint wrist_right_ft_tool_link_42693_right_46739_joint: type fixed, parent wrist_right_ft_tool_link_42693, child right_46739, origin xyz=0.016 -5.877128e-08 0 rpy=-2.356193 1.5707923 0.78539306
- joint arm_left_1_joint: child TIAGo_left_arm_44027 -> TIAGo_left_arm_43980; parent TIAGo left arm_44012 -> TIAGo left arm_43965
- joint arm_left_2_joint: child arm_left_2_link_44060 -> arm_left_2_link_44013; parent TIAGo_left_arm_44027 -> TIAGo_left_arm_43980
- joint arm_left_3_joint: child arm_left_3_link_44074 -> arm_left_3_link_44027; parent arm_left_2_link_44060 -> arm_left_2_link_44013
- joint arm_left_4_joint: child arm_left_4_link_44108 -> arm_left_4_link_44061; parent arm_left_3_link_44074 -> arm_left_3_link_44027
- joint arm_left_5_joint: child arm_left_5_link_44142 -> arm_left_5_link_44095; parent arm_left_4_link_44108 -> arm_left_4_link_44061
- joint arm_left_6_joint: child arm_left_6_link_44157 -> arm_left_6_link_44110; parent arm_left_5_link_44142 -> arm_left_5_link_44095
- joint arm_left_7_joint: child arm_left_7_link_44172 -> arm_left_7_link_44125; parent arm_left_6_link_44157 -> arm_left_6_link_44110
- joint arm_right_1_joint: child TIAGo_right_arm_42582 -> TIAGo_right_arm_42535; parent TIAGo right arm_42567 -> TIAGo right arm_42520
- joint arm_right_2_joint: child arm_right_2_link_42616 -> arm_right_2_link_42569; parent TIAGo_right_arm_42582 -> TIAGo_right_arm_42535
- joint arm_right_3_joint: child arm_right_3_link_42630 -> arm_right_3_link_42583; parent arm_right_2_link_42616 -> arm_right_2_link_42569
- joint arm_right_4_joint: child arm_right_4_link_42664 -> arm_right_4_link_42617; parent arm_right_3_link_42630 -> arm_right_3_link_42583
- joint arm_right_5_joint: child arm_right_5_link_42698 -> arm_right_5_link_42651; parent arm_right_4_link_42664 -> arm_right_4_link_42617
- joint arm_right_6_joint: child arm_right_6_link_42713 -> arm_right_6_link_42666; parent arm_right_5_link_42698 -> arm_right_5_link_42651
- joint arm_right_7_joint: child arm_right_7_link_42728 -> arm_right_7_link_42681; parent arm_right_6_link_42713 -> arm_right_6_link_42666
- joint left_hand_gripper_left_finger_joint: child gripper_left_finger_link_49229 -> gripper_left_finger_link_49182; parent left_48701 -> left_48654
- joint left_hand_gripper_right_finger_joint: child gripper_right_finger_link_49262 -> gripper_right_finger_link_49215; parent left_48701 -> left_48654
- joint right_hand_gripper_left_finger_joint: child gripper_left_finger_link_47314 -> gripper_left_finger_link_47267; parent right_46786 -> right_46739
- joint right_hand_gripper_right_finger_joint: child gripper_right_finger_link_47347 -> gripper_right_finger_link_47300; parent right_46786 -> right_46739

File: tests/api/controllers/robot_urdf/ur5e_reference.urdf (robot description, URDF)
Before this commit: robot UR5e, 8 links, 7 joints
Links:
- removed link track_354
- added link track_307
Joints:
- removed joint wrist_3_link_track_354_joint
- added joint wrist_3_link_track_307_joint: type fixed, parent wrist_3_link, child track_307, origin xyz=0 0.1 0 rpy=0 0 0
