Commit message: Add changelog

File: tests/api/controllers/robot_urdf/prob3_reference.urdf (robot description, URDF)
Before this commit: robot P-Rob3, 19 links, 18 joints
Links:
- added link gripper middle distance sensor
- added link left finger sensor 0
- added link left finger sensor 1
- added link left finger sensor 2
- added link left finger sensor 3
- added link right finger sensor 0
- added link right finger sensor 1
- added link right finger sensor 2
- added link right finger sensor 3
- added link ts_emitter
Joints:
- added joint left finger_50285_left finger sensor 0_joint: type fixed, parent left finger_50285, child left finger sensor 0, origin xyz=0.013 0.02 0.118 rpy=0 0 0
- added joint left finger_50285_left finger sensor 1_joint: type fixed, parent left finger_50285, child left finger sensor 1, origin xyz=-0.013 0.02 0.118 rpy=0 0 3.1415927
- added joint left finger_50285_left finger sensor 2_joint: type fixed, parent left finger_50285, child left finger sensor 2, origin xyz=-7.548e-10 0.0214379 0.13449 rpy=-3.3035767e-06 -1.1257437 -1.5707953
- added joint left finger_50285_left finger sensor 3_joint: type fixed, parent left finger_50285, child left finger sensor 3, origin xyz=-6.75982e-08 0.0173238 0.0871813 rpy=7.8457396e-07 0.26179942 1.5708023
- added joint link_6_top_ts_emitter_joint: type fixed, parent link_6_top, child ts_emitter, origin xyz=0 0 0.02075 rpy=0 0 0
- added joint link_base_tcp180_50200_gripper middle distance sensor_joint: type fixed, parent link_base_tcp180_50200, child gripper middle distance sensor, origin xyz=0 0 0.085 rpy=0 -1.5707897 0
- added joint right finger_50237_right finger sensor 0_joint: type fixed, parent right finger_50237, child right finger sensor 0, origin xyz=0.013 0.02 0.118 rpy=0 0 0
- added joint right finger_50237_right finger sensor 1_joint: type fixed, parent right finger_50237, child right finger sensor 1, origin xyz=-0.013 0.02 0.118 rpy=0 0 3.1415927
- added joint right finger_50237_right finger sensor 2_joint: type fixed, parent right finger_50237, child right finger sensor 2, origin xyz=-7.548e-10 0.0214379 0.13449 rpy=-3.3035767e-06 -1.1257437 -1.5707953
- added joint right finger_50237_right finger sensor 3_joint: type fixed, parent right finger_50237, child right finger sensor 3, origin xyz=-6.75982e-08 0.0173238 0.0871813 rpy=7.8457396e-07 0.26179942 1.5708023
- joint link_6_top_link_base_tcp180_50200_joint: origin xyz=0 0 0.0985 rpy=0 0 0 -> xyz=0 0 0.07775 rpy=0 0 0

File: tests/api/controllers/robot_urdf/tiago_reference.urdf (robot description, URDF)
Before this commit: robot TIAGo++, 84 links, 83 joints
Links:
- added link accelerometer
- added link gyro
- added link inertial unit
- added link ts_emitter
Joints:
- added joint base_link_accelerometer_joint: type fixed, parent base_link, child accelerometer, origin xyz=0 0 0 rpy=0 0 0
- added joint base_link_gyro_joint: type fixed, parent base_link, child gyro, origin xyz=0 0 0 rpy=0 0 0
- added joint base_link_inertial unit_joint: type fixed, parent base_link, child inertial unit, origin xyz=0 0 0 rpy=0 0 0
- added joint head_2_link_ts_emitter_joint: type fixed, parent head_2_link, child ts_emitter, origin xyz=0.107 0.0802 0 rpy=0 0 0

File: tests/api/controllers/robot_urdf/ur5e_reference.urdf (robot description, URDF)
Before this commit: robot UR5e, 8 links, 7 joints
Links:
- added link ts_emitter
Joints:
- added joint wrist_3_link_ts_emitter_joint: type fixed, parent wrist_3_link, child ts_emitter, origin xyz=0 0.1 0 rpy=0 0 0

Commit message: Fixed robot_urdf test on Windows

File: tests/api/controllers/robot_urdf/prob3_reference.urdf (robot description, URDF)
Before this commit: robot P-Rob3, 29 links, 28 joints
Joints:
- joint 7 left: axis -1 -2.614661e-06 4.528642e-07 -> -1 -0.000003 0; origin xyz=0 0 0.058 rpy=0.3430009 4.528642e-07 3.14159 -> xyz=0 0 0.058 rpy=0.343001 0 3.14159
- joint base_link_cap screw_joint: origin xyz=0.0962 0 0.099 rpy=3.1415927 -1.5707923 3.1415927 -> xyz=0.0962 0 0.099 rpy=3.141593 -1.570792 3.141593
- joint left finger_left finger sensor 1_joint: origin xyz=-0.013 0.02 0.118 rpy=0 0 3.1415927 -> xyz=-0.013 0.02 0.118 rpy=0 0 3.141593
- joint left finger_left finger sensor 2_joint: origin xyz=-7.548e-10 0.0214379 0.13449 rpy=-3.3035767e-06 -1.1257437 -1.5707953 -> xyz=-0 0.021438 0.13449 rpy=-0.000003 -1.125744 -1.570795
- joint left finger_left finger sensor 3_joint: origin xyz=-6.75982e-08 0.0173238 0.0871813 rpy=7.8457396e-07 0.26179942 1.5708023 -> xyz=-0 0.017324 0.087181 rpy=0.000001 0.261799 1.570802
- joint link_6_top_button 0_joint: origin xyz=-0.0501799 0.0432036 0.0089 rpy=0 0 0.9162997 -> xyz=-0.05018 0.043204 0.0089 rpy=0 0 0.9163
- joint link_6_top_button 1_joint: origin xyz=-0.0643129 0.0151085 0.0089 rpy=0 0 1.3090003 -> xyz=-0.064313 0.015109 0.0089 rpy=0 0 1.309
- joint link_6_top_button 2_joint: origin xyz=-0.0642012 -0.0156443 0.0089 rpy=0 0 1.8 -> xyz=-0.064201 -0.015644 0.0089 rpy=0 0 1.8
- joint link_6_top_button 3_joint: origin xyz=-0.0505297 -0.0431944 0.0089 rpy=0 0 2.28 -> xyz=-0.05053 -0.043194 0.0089 rpy=0 0 2.28
- joint link_6_top_button 4_joint: origin xyz=0.0502593 -0.0432647 0.0089 rpy=0 0 0.9162997 -> xyz=0.050259 -0.043265 0.0089 rpy=0 0 0.9163
- joint link_6_top_button 5_joint: origin xyz=0.064216 -0.0150831 0.0089 rpy=0 0 1.3090003 -> xyz=0.064216 -0.015083 0.0089 rpy=0 0 1.309
- joint link_6_top_button 6_joint: origin xyz=0.0642009 0.0156447 0.0089 rpy=0 0 1.8 -> xyz=0.064201 0.015645 0.0089 rpy=0 0 1.8
- joint link_6_top_button 7_joint: origin xyz=0.0503023 0.042999 0.0089 rpy=0 0 2.28 -> xyz=0.050302 0.042999 0.0089 rpy=0 0 2.28
- joint link_base_tcp180_gripper middle distance sensor_joint: origin xyz=0 0 0.085 rpy=0 -1.5707897 0 -> xyz=0 0 0.085 rpy=0 -1.57079 0
- joint right finger_right finger sensor 1_joint: origin xyz=-0.013 0.02 0.118 rpy=0 0 3.1415927 -> xyz=-0.013 0.02 0.118 rpy=0 0 3.141593
- joint right finger_right finger sensor 2_joint: origin xyz=-7.548e-10 0.0214379 0.13449 rpy=-3.3035767e-06 -1.1257437 -1.5707953 -> xyz=-0 0.021438 0.13449 rpy=-0.000003 -1.125744 -1.570795
- joint right finger_right finger sensor 3_joint: origin xyz=-6.75982e-08 0.0173238 0.0871813 rpy=7.8457396e-07 0.26179942 1.5708023 -> xyz=-0 0.017324 0.087181 rpy=0.000001 0.261799 1.570802

File: tests/api/controllers/robot_urdf/tiago_reference.urdf (robot description, URDF)
Before this commit: robot TIAGo++, 89 links, 88 joints
Joints:
- joint SMALL_WHEEL_JOINT: axis 0 -3.6732051e-06 1 -> 0 -0.000004 1
- joint SMALL_WHEEL_JOINT_0: axis 0 -3.6732051e-06 1 -> 0 -0.000004 1
- joint SMALL_WHEEL_JOINT_1: axis 0 -3.6732051e-06 1 -> 0 -0.000004 1
- joint SMALL_WHEEL_JOINT_2: axis 0 -3.6732051e-06 1 -> 0 -0.000004 1
- joint arm_left_2_joint: axis 0 -3.6732051e-06 -1 -> 0 -0.000004 -1
- joint arm_left_3_joint: axis -6.056618e-05 -6.055936e-05 -1 -> -0.000061 -0.000061 -1; origin xyz=0.0895 5.5098077e-09 -1.0118208e-14 rpy=1.5708569 -0.0001126458 -1.5708569 -> xyz=0.0895 0 -0 rpy=1.570857 -0.000113 -1.570857
- joint arm_left_4_joint: axis 2.8276386e-06 -2.8276306e-06 1 -> 0.000003 -0.000003 1; origin xyz=-0.01999986 -0.026999861 -0.2197 rpy=2.356193 -1.5707923 2.356193 -> xyz=-0.02 -0.027 -0.2197 rpy=2.356193 -1.570792 2.356193
- joint arm_left_5_joint: axis -3.6732051e-06 0 -1 -> -0.000004 0 -1; origin xyz=-0.162 0.02 0.027 rpy=3.1415927 -1.5707927 3.1415927 -> xyz=-0.162 0.02 0.027 rpy=3.141593 -1.570793 3.141593
- joint arm_left_6_joint: axis -2.8276386e-06 2.8276306e-06 -1 -> -0.000003 0.000003 -1; origin xyz=0 0 0.15 rpy=2.356193 -1.5707923 2.356193 -> xyz=0 0 0.15 rpy=2.356193 -1.570792 2.356193
- joint arm_left_7_joint: axis 2.8276306e-06 -2.8276386e-06 -1 -> 0.000003 -0.000003 -1; origin xyz=0 0 0 rpy=1.5707991 -2.8276386e-06 1.5707991 -> xyz=0 0 0 rpy=1.570799 -0.000003 1.570799
- joint arm_left_7_link_wrist_left_ft_tool_link_joint: origin xyz=-1.5551969e-07 1.5552013e-07 0.067725 rpy=2.356193 -1.5707923 2.356193 -> xyz=-0 0 0.067725 rpy=2.356193 -1.570792 2.356193
- joint arm_right_2_joint: axis 0 3.6732051e-06 1 -> 0 0.000004 1
- joint arm_right_3_joint: axis -2.8276306e-06 2.8276386e-06 1 -> -0.000003 0.000003 1; origin xyz=0.0895 5.5098077e-09 -1.0118208e-14 rpy=1.5707991 -2.8276386e-06 1.5707991 -> xyz=0.0895 0 -0 rpy=1.570799 -0.000003 1.570799
- joint arm_right_4_joint: axis 2.8276386e-06 2.8276306e-06 -1 -> 0.000003 0.000003 -1; origin xyz=0.020000502 0.0014995021 -0.3991 rpy=2.356193 1.5707923 -2.356193 -> xyz=0.020001 0.0015 -0.3991 rpy=2.356193 1.570792 -2.356193
- joint arm_right_5_joint: axis 1.349254e-11 5.1946963e-06 1 -> 0 0.000005 1; origin xyz=0.16300008 0.020000074 0.001 rpy=-1.5707937 -1.5707911 -1.5707937 -> xyz=0.163 0.02 0.001 rpy=-1.570794 -1.570791 -1.570794
- joint arm_right_6_joint: axis 2.8276386e-06 2.8276306e-06 -1 -> 0.000003 0.000003 -1; origin xyz=0 0 0.15 rpy=2.356193 1.5707923 -2.356193 -> xyz=0 0 0.15 rpy=2.356193 1.570792 -2.356193
- joint arm_right_7_joint: axis 2.8276306e-06 -2.8276386e-06 1 -> 0.000003 -0.000003 1; origin xyz=0 0 0 rpy=-1.5707991 2.8276386e-06 1.5707991 -> xyz=0 0 0 rpy=-1.570799 0.000003 1.570799
- joint arm_right_7_link_wrist_right_ft_tool_link_joint: origin xyz=1.5551969e-07 -1.5552013e-07 0.067725 rpy=2.356193 -1.5707923 2.356193 -> xyz=0 -0 0.067725 rpy=2.356193 -1.570792 2.356193
- joint base_link_Hokuyo URG-04LX-UG01_joint: origin xyz=0.202 0 -0.004 rpy=1.5707414 0.00011829441 -1.5707414 -> xyz=0.202 0 -0.004 rpy=1.570741 0.000118 -1.570741
- joint base_link_base_sonar_01_link_joint: origin xyz=-0.183 -0.183 0.1728 rpy=0 0 -2.3561852 -> xyz=-0.183 -0.183 0.1728 rpy=0 0 -2.356185
- joint base_link_base_sonar_02_link_joint: origin xyz=-0.259 0 0.173 rpy=0 0 -3.1415854 -> xyz=-0.259 0 0.173 rpy=0 0 -3.141585
- joint head_2_joint: axis 0 3.6732051e-06 1 -> 0 0.000004 1
- joint left_cap screw(1)_joint: origin xyz=0.0477 0.008 -0.043 rpy=3.1415927 -1.5707927 3.1415927 -> xyz=0.0477 0.008 -0.043 rpy=3.141593 -1.570793 3.141593
- joint left_cap screw(10)_joint: origin xyz=-0.0477 -0.008 -0.043 rpy=3.1415927 1.5707927 3.1415927 -> xyz=-0.0477 -0.008 -0.043 rpy=3.141593 1.570793 3.141593
- joint left_cap screw(11)_joint: origin xyz=-0.0477 -0.008 -0.0108 rpy=3.1415927 1.5707927 3.1415927 -> xyz=-0.0477 -0.008 -0.0108 rpy=3.141593 1.570793 3.141593
- joint left_cap screw(2)_joint: origin xyz=0.0477 0.008 -0.075 rpy=3.1415927 -1.5707927 3.1415927 -> xyz=0.0477 0.008 -0.075 rpy=3.141593 -1.570793 3.141593
- joint left_cap screw(3)_joint: origin xyz=0.0477 -0.008 -0.075 rpy=3.1415927 -1.5707927 3.1415927 -> xyz=0.0477 -0.008 -0.075 rpy=3.141593 -1.570793 3.141593
- joint left_cap screw(4)_joint: origin xyz=0.0477 -0.008 -0.043 rpy=3.1415927 -1.5707927 3.1415927 -> xyz=0.0477 -0.008 -0.043 rpy=3.141593 -1.570793 3.141593
- joint left_cap screw(5)_joint: origin xyz=0.0477 -0.008 -0.0108 rpy=3.1415927 -1.5707927 3.1415927 -> xyz=0.0477 -0.008 -0.0108 rpy=3.141593 -1.570793 3.141593
- joint left_cap screw(6)_joint: origin xyz=-0.0477 0.008 -0.0108 rpy=3.1415927 1.5707927 3.1415927 -> xyz=-0.0477 0.008 -0.0108 rpy=3.141593 1.570793 3.141593
- joint left_cap screw(7)_joint: origin xyz=-0.0477 0.008 -0.043 rpy=3.1415927 1.5707927 3.1415927 -> xyz=-0.0477 0.008 -0.043 rpy=3.141593 1.570793 3.141593
- joint left_cap screw(8)_joint: origin xyz=-0.0477 0.008 -0.075 rpy=3.1415927 1.5707927 3.1415927 -> xyz=-0.0477 0.008 -0.075 rpy=3.141593 1.570793 3.141593
- joint left_cap screw(9)_joint: origin xyz=-0.0477 -0.008 -0.075 rpy=3.1415927 1.5707927 3.1415927 -> xyz=-0.0477 -0.008 -0.075 rpy=3.141593 1.570793 3.141593
- joint left_cap screw_joint: origin xyz=0.0477 0.008 -0.0108 rpy=3.1415927 -1.5707927 3.1415927 -> xyz=0.0477 0.008 -0.0108 rpy=3.141593 -1.570793 3.141593
- joint left_hand_gripper_left_finger_joint: axis 1 9.265359e-05 0 -> 1 0.000093 0
- joint right_cap screw(1)_23_joint: origin xyz=0.0477 0.008 -0.043 rpy=3.1415927 -1.5707927 3.1415927 -> xyz=0.0477 0.008 -0.043 rpy=3.141593 -1.570793 3.141593
- joint right_cap screw(10)_14_joint: origin xyz=-0.0477 -0.008 -0.043 rpy=3.1415927 1.5707927 3.1415927 -> xyz=-0.0477 -0.008 -0.043 rpy=3.141593 1.570793 3.141593
- joint right_cap screw(11)_13_joint: origin xyz=-0.0477 -0.008 -0.0108 rpy=3.1415927 1.5707927 3.1415927 -> xyz=-0.0477 -0.008 -0.0108 rpy=3.141593 1.570793 3.141593
- joint right_cap screw(2)_22_joint: origin xyz=0.0477 0.008 -0.075 rpy=3.1415927 -1.5707927 3.1415927 -> xyz=0.0477 0.008 -0.075 rpy=3.141593 -1.570793 3.141593
- joint right_cap screw(3)_21_joint: origin xyz=0.0477 -0.008 -0.075 rpy=3.1415927 -1.5707927 3.1415927 -> xyz=0.0477 -0.008 -0.075 rpy=3.141593 -1.570793 3.141593
- joint right_cap screw(4)_20_joint: origin xyz=0.0477 -0.008 -0.043 rpy=3.1415927 -1.5707927 3.1415927 -> xyz=0.0477 -0.008 -0.043 rpy=3.141593 -1.570793 3.141593
- joint right_cap screw(5)_19_joint: origin xyz=0.0477 -0.008 -0.0108 rpy=3.1415927 -1.5707927 3.1415927 -> xyz=0.0477 -0.008 -0.0108 rpy=3.141593 -1.570793 3.141593
- joint right_cap screw(6)_18_joint: origin xyz=-0.0477 0.008 -0.0108 rpy=3.1415927 1.5707927 3.1415927 -> xyz=-0.0477 0.008 -0.0108 rpy=3.141593 1.570793 3.141593
- joint right_cap screw(7)_17_joint: origin xyz=-0.0477 0.008 -0.043 rpy=3.1415927 1.5707927 3.1415927 -> xyz=-0.0477 0.008 -0.043 rpy=3.141593 1.570793 3.141593
- joint right_cap screw(8)_16_joint: origin xyz=-0.0477 0.008 -0.075 rpy=3.1415927 1.5707927 3.1415927 -> xyz=-0.0477 0.008 -0.075 rpy=3.141593 1.570793 3.141593
- joint right_cap screw(9)_15_joint: origin xyz=-0.0477 -0.008 -0.075 rpy=3.1415927 1.5707927 3.1415927 -> xyz=-0.0477 -0.008 -0.075 rpy=3.141593 1.570793 3.141593
- joint right_cap screw_24_joint: origin xyz=0.0477 0.008 -0.0108 rpy=3.1415927 -1.5707927 3.1415927 -> xyz=0.0477 0.008 -0.0108 rpy=3.141593 -1.570793 3.141593
- joint right_hand_gripper_left_finger_joint: axis 1 9.265359e-05 0 -> 1 0.000093 0
- joint torso_lift_link_TIAGo right arm_joint: origin xyz=1.3492402e-12 -3.6732052e-07 0 rpy=0 0 4.6928203e-06 -> xyz=0 -0 0 rpy=0 0 0.000005
- joint wheel_left_joint: axis 0 -3.6732051e-06 -1 -> 0 -0.000004 -1
- joint wheel_right_joint: axis 0 -3.6732051e-06 -1 -> 0 -0.000004 -1
- joint wrist_left_ft_tool_link_left_joint: origin xyz=0.016 -5.877128e-08 0 rpy=-2.356193 1.5707923 0.78539306 -> xyz=0.016 -0 0 rpy=-2.356193 1.570792 0.785393
- joint wrist_right_ft_tool_link_right_joint: origin xyz=0.016 -5.877128e-08 0 rpy=-2.356193 1.5707923 0.78539306 -> xyz=0.016 -0 0 rpy=-2.356193 1.570792 0.785393

Commit message: Fixed reference URDF files

File: tests/api/controllers/robot_urdf/prob3_reference.urdf (robot description, URDF)
Before this commit: robot P-Rob3, 29 links, 28 joints
Joints:
- joint left finger_left finger sensor 2_joint: origin xyz=-0 0.021438 0.13449 rpy=-0.000003 -1.125744 -1.570795 -> xyz=0 0.021438 0.13449 rpy=-0.000003 -1.125744 -1.570795
- joint left finger_left finger sensor 3_joint: origin xyz=-0 0.017324 0.087181 rpy=0.000001 0.261799 1.570802 -> xyz=0 0.017324 0.087181 rpy=0.000001 0.261799 1.570802
- joint right finger_right finger sensor 2_joint: origin xyz=-0 0.021438 0.13449 rpy=-0.000003 -1.125744 -1.570795 -> xyz=0 0.021438 0.13449 rpy=-0.000003 -1.125744 -1.570795
- joint right finger_right finger sensor 3_joint: origin xyz=-0 0.017324 0.087181 rpy=0.000001 0.261799 1.570802 -> xyz=0 0.017324 0.087181 rpy=0.000001 0.261799 1.570802

File: tests/api/controllers/robot_urdf/tiago_reference.urdf (robot description, URDF)
Before this commit: robot TIAGo++, 89 links, 88 joints
Joints:
- joint arm_left_3_joint: origin xyz=0.0895 0 -0 rpy=1.570857 -0.000113 -1.570857 -> xyz=0.0895 0 0 rpy=1.570857 -0.000113 -1.570857
- joint arm_left_7_link_wrist_left_ft_tool_link_joint: origin xyz=-0 0 0.067725 rpy=2.356193 -1.570792 2.356193 -> xyz=0 0 0.067725 rpy=2.356193 -1.570792 2.356193
- joint arm_right_3_joint: origin xyz=0.0895 0 -0 rpy=1.570799 -0.000003 1.570799 -> xyz=0.0895 0 0 rpy=1.570799 -0.000003 1.570799
- joint arm_right_7_link_wrist_right_ft_tool_link_joint: origin xyz=0 -0 0.067725 rpy=2.356193 -1.570792 2.356193 -> xyz=0 0 0.067725 rpy=2.356193 -1.570792 2.356193
- joint torso_lift_link_TIAGo right arm_joint: origin xyz=0 -0 0 rpy=0 0 0.000005 -> xyz=0 0 0 rpy=0 0 0.000005
- joint wrist_left_ft_tool_link_left_joint: origin xyz=0.016 -0 0 rpy=-2.356193 1.570792 0.785393 -> xyz=0.016 0 0 rpy=-2.356193 1.570792 0.785393
- joint wrist_right_ft_tool_link_right_joint: origin xyz=0.016 -0 0 rpy=-2.356193 1.570792 0.785393 -> xyz=0.016 0 0 rpy=-2.356193 1.570792 0.785393

Commit message: tests and protos until supervisor_export_image.wbt

File: tests/api/controllers/robot_urdf/prob3_reference.urdf (robot description, URDF)
Before this commit: robot P-Rob3, 29 links, 28 joints
Joints:
- joint link_6_top_button 0_joint: origin xyz=-0.05018 0.043204 0.0089 rpy=0 0 0.9163 -> xyz=-0.05018 0.043204 0.0089 rpy=-1.570796 0 0.9163
- joint link_6_top_button 1_joint: origin xyz=-0.064313 0.015109 0.0089 rpy=0 0 1.309 -> xyz=-0.064313 0.015109 0.0089 rpy=-1.570796 0 1.309
- joint link_6_top_button 2_joint: origin xyz=-0.064201 -0.015644 0.0089 rpy=0 0 1.8 -> xyz=-0.064201 -0.015644 0.0089 rpy=-1.570796 0 1.8
- joint link_6_top_button 3_joint: origin xyz=-0.05053 -0.043194 0.0089 rpy=0 0 2.28 -> xyz=-0.05053 -0.043194 0.0089 rpy=-1.570796 0 2.28
- joint link_6_top_button 4_joint: origin xyz=0.050259 -0.043265 0.0089 rpy=0 0 0.9163 -> xyz=0.050259 -0.043265 0.0089 rpy=-1.570796 0 0.9163
- joint link_6_top_button 5_joint: origin xyz=0.064216 -0.015083 0.0089 rpy=0 0 1.309 -> xyz=0.064216 -0.015083 0.0089 rpy=-1.570796 0 1.309
- joint link_6_top_button 6_joint: origin xyz=0.064201 0.015645 0.0089 rpy=0 0 1.8 -> xyz=0.064201 0.015645 0.0089 rpy=-1.570796 0 1.8
- joint link_6_top_button 7_joint: origin xyz=0.050302 0.042999 0.0089 rpy=0 0 2.28 -> xyz=0.050302 0.042999 0.0089 rpy=-1.570796 0 2.28

Commit message: Fix capscrew in p-rob3

File: tests/api/controllers/robot_urdf/prob3_reference.urdf (robot description, URDF)
Before this commit: robot P-Rob3, 29 links, 28 joints
Joints:
- joint base_link_cap screw_joint: origin xyz=0.0962 0 0.099 rpy=3.141593 -1.570792 3.141593 -> xyz=0.0962 0 0.099 rpy=0 0 3.141593
