Commit message: ENU/FLU Conversion Plan (#3073)
* Convert humanoid_sprint

* convert camera_motion_blur

* convert led

* convert compass

* conert force_3d_sensor

* Convert factory

* convert force_sensor

* convert pen, altimeter, hinge_2_joint, encoders

* small fix accelerometer

* 2

* FLU: convert objects/road (#3646)

* init

* Convert Road & CrashBarrier

* Convert LaneSeparation and Fix barriers/borders

* Convert RoadIntersection

* Swap Road coordinates

* Swap StraightRoadSegment coordinates

* Convert CurvedRoadSegment and HelicoidalRoadSegment

* Swap coordinates in LaneSeparation and RoadIntersection

* Swap coordinates in AddLaneRoadSegment and AddLanesRoadSegment

* Convert Crossroad

* Convert RoadPillar

* Undo LateSeparation changes

* Undo LateSeparation changes

* Convert Roundabout

* Convert CrossRoad

* Convert CrossRoad shapes in worlds

* Fix Roundabout

* Functional CrashBarrier (still broken with subdivision != 0)

* Finalize

* Cleanup

* Fix

* Fix `StraightStairs` and tiago++ world (#3747)

* Fix stairs texture

* Fix tiago++.wbt

* Apply suggestions from code review

Co-authored-by: Benjamin Délèze <benjamin.deleze@epfl.ch>

* convert camera

* FLU hoap mavic summit mindstorms (#3721)

* hoap2

* hoap2 inertiaMatrix

* hoap2 worlds

* mavic

* mavic controller

* mavic world

* summitxls

* correct friction

* lidars position

* revert friction

* revert friction change

* summitXL world

* mindstorms

* rover.wbt

* fabtino

* fabtino.wbt

* doc

* update robotino3_platform

* mavic road

* Update projects/robots/fujitsu/hoap2/protos/Hoap2.proto

Co-authored-by: ad-daniel <44834743+ad-daniel@users.noreply.github.com>

* Update projects/robots/fujitsu/hoap2/protos/Hoap2.proto

Co-authored-by: ad-daniel <44834743+ad-daniel@users.noreply.github.com>

* Update projects/robots/fujitsu/hoap2/protos/Hoap2.proto

Co-authored-by: ad-daniel <44834743+ad-daniel@users.noreply.github.com>

* Update projects/robots/fujitsu/hoap2/protos/Hoap2.proto

Co-authored-by: ad-daniel <44834743+ad-daniel@users.noreply.github.com>

* Update projects/robots/fujitsu/hoap2/protos/Hoap2.proto

Co-authored-by: ad-daniel <44834743+ad-daniel@users.noreply.github.com>

* Update projects/robots/fujitsu/hoap2/protos/Hoap2.proto

Co-authored-by: ad-daniel <44834743+ad-daniel@users.noreply.github.com>

* Update projects/robots/dji/mavic/worlds/mavic_2_pro.wbt

Co-authored-by: ad-daniel <44834743+ad-daniel@users.noreply.github.com>

* Update projects/robots/dji/mavic/worlds/mavic_2_pro.wbt

Co-authored-by: ad-daniel <44834743+ad-daniel@users.noreply.github.com>

* Update projects/robots/dji/mavic/worlds/mavic_2_pro.wbt

Co-authored-by: ad-daniel <44834743+ad-daniel@users.noreply.github.com>

* Update projects/robots/dji/mavic/worlds/mavic_2_pro.wbt

Co-authored-by: ad-daniel <44834743+ad-daniel@users.noreply.github.com>

* Update projects/robots/dji/mavic/worlds/mavic_2_pro.wbt

Co-authored-by: ad-daniel <44834743+ad-daniel@users.noreply.github.com>

* Update projects/robots/fujitsu/hoap2/protos/Hoap2.proto

Co-authored-by: ad-daniel <44834743+ad-daniel@users.noreply.github.com>

* Update projects/robots/fujitsu/hoap2/protos/Hoap2.proto

Co-authored-by: ad-daniel <44834743+ad-daniel@users.noreply.github.com>

* Update projects/robots/fujitsu/hoap2/protos/Hoap2.proto

Co-authored-by: ad-daniel <44834743+ad-daniel@users.noreply.github.com>

* Update projects/robots/fujitsu/hoap2/protos/Hoap2.proto

Co-authored-by: ad-daniel <44834743+ad-daniel@users.noreply.github.com>

* Update projects/robots/fujitsu/hoap2/worlds/hoap2_sumo.wbt

Co-authored-by: ad-daniel <44834743+ad-daniel@users.noreply.github.com>

* Update projects/robots/fujitsu/hoap2/worlds/hoap2_sumo.wbt

Co-authored-by: ad-daniel <44834743+ad-daniel@users.noreply.github.com>

* Update projects/robots/lego/mindstorms/worlds/rover.wbt

Co-authored-by: ad-daniel <44834743+ad-daniel@users.noreply.github.com>

* Update projects/robots/rec/fabtino/worlds/fabtino.wbt

Co-authored-by: ad-daniel <44834743+ad-daniel@users.noreply.github.com>

* Update projects/robots/rec/fabtino/worlds/fabtino.wbt

Co-authored-by: ad-daniel <44834743+ad-daniel@users.noreply.github.com>

* Update projects/robots/rec/fabtino/worlds/fabtino.wbt

Co-authored-by: ad-daniel <44834743+ad-daniel@users.noreply.github.com>

* Update projects/robots/rec/fabtino/worlds/fabtino.wbt

Co-authored-by: ad-daniel <44834743+ad-daniel@users.noreply.github.com>

* Update projects/robots/rec/fabtino/worlds/fabtino.wbt

Co-authored-by: ad-daniel <44834743+ad-daniel@users.noreply.github.com>

* Update projects/robots/rec/fabtino/worlds/fabtino.wbt

Co-authored-by: ad-daniel <44834743+ad-daniel@users.noreply.github.com>

* Update projects/robots/rec/fabtino/worlds/fabtino.wbt

Co-authored-by: ad-daniel <44834743+ad-daniel@users.noreply.github.com>

* Update projects/robots/rec/fabtino/worlds/fabtino.wbt

Co-authored-by: ad-daniel <44834743+ad-daniel@users.noreply.github.com>

* Update projects/robots/rec/fabtino/worlds/fabtino.wbt

Co-authored-by: ad-daniel <44834743+ad-daniel@users.noreply.github.com>

* Update projects/robots/rec/fabtino/worlds/fabtino.wbt

Co-authored-by: ad-daniel <44834743+ad-daniel@users.noreply.github.com>

* Update projects/robots/rec/fabtino/worlds/fabtino.wbt

Co-authored-by: ad-daniel <44834743+ad-daniel@users.noreply.github.com>

* Update projects/robots/rec/fabtino/worlds/fabtino.wbt

Co-authored-by: ad-daniel <44834743+ad-daniel@users.noreply.github.com>

* Update projects/robots/rec/fabtino/worlds/fabtino.wbt

Co-authored-by: ad-daniel <44834743+ad-daniel@users.noreply.github.com>

* Update projects/robots/robotnik/summit_xl_steel/worlds/summit_xl_steel.wbt

Co-authored-by: ad-daniel <44834743+ad-daniel@users.noreply.github.com>

* Update projects/robots/robotnik/summit_xl_steel/worlds/summit_xl_steel.wbt

Co-authored-by: ad-daniel <44834743+ad-daniel@users.noreply.github.com>

* Update projects/robots/robotnik/summit_xl_steel/worlds/summit_xl_steel.wbt

Co-authored-by: ad-daniel <44834743+ad-daniel@users.noreply.github.com>

* Update projects/robots/robotnik/summit_xl_steel/worlds/summit_xl_steel.wbt

Co-authored-by: ad-daniel <44834743+ad-daniel@users.noreply.github.com>

* Update projects/robots/robotnik/summit_xl_steel/worlds/summit_xl_steel.wbt

Co-authored-by: ad-daniel <44834743+ad-daniel@users.noreply.github.com>

* Update projects/robots/robotnik/summit_xl_steel/worlds/summit_xl_steel.wbt

Co-authored-by: ad-daniel <44834743+ad-daniel@users.noreply.github.com>

* Update projects/robots/robotnik/summit_xl_steel/worlds/summit_xl_steel.wbt

Co-authored-by: ad-daniel <44834743+ad-daniel@users.noreply.github.com>

* Update projects/robots/robotnik/summit_xl_steel/worlds/summit_xl_steel.wbt

Co-authored-by: ad-daniel <44834743+ad-daniel@users.noreply.github.com>

* Update projects/robots/robotnik/summit_xl_steel/worlds/summit_xl_steel.wbt

Co-authored-by: ad-daniel <44834743+ad-daniel@users.noreply.github.com>

* Update projects/robots/robotnik/summit_xl_steel/worlds/summit_xl_steel.wbt

Co-authored-by: ad-daniel <44834743+ad-daniel@users.noreply.github.com>

* Update projects/robots/robotnik/summit_xl_steel/worlds/summit_xl_steel.wbt

Co-authored-by: ad-daniel <44834743+ad-daniel@users.noreply.github.com>

* Update projects/robots/robotnik/summit_xl_steel/worlds/summit_xl_steel.wbt

Co-authored-by: ad-daniel <44834743+ad-daniel@users.noreply.github.com>

* Update projects/robots/robotnik/summit_xl_steel/worlds/summit_xl_steel.wbt

Co-authored-by: ad-daniel <44834743+ad-daniel@users.noreply.github.com>

* Update projects/robots/robotnik/summit_xl_steel/worlds/summit_xl_steel.wbt

Co-authored-by: ad-daniel <44834743+ad-daniel@users.noreply.github.com>

* Update projects/robots/robotnik/summit_xl_steel/worlds/summit_xl_steel.wbt

Co-authored-by: ad-daniel <44834743+ad-daniel@users.noreply.github.com>

* Update projects/robots/robotnik/summit_xl_steel/worlds/summit_xl_steel.wbt

Co-authored-by: ad-daniel <44834743+ad-daniel@users.noreply.github.com>

* Update projects/robots/robotnik/summit_xl_steel/worlds/summit_xl_steel.wbt

Co-authored-by: ad-daniel <44834743+ad-daniel@users.noreply.github.com>

* Update projects/robots/dji/mavic/worlds/mavic_2_pro.wbt

Co-authored-by: ad-daniel <44834743+ad-daniel@users.noreply.github.com>

* correct translation for plateform

Co-authored-by: ad-daniel <44834743+ad-daniel@users.noreply.github.com>

* convert camera_auto_focus

* camera with camera issue

* spherical_camera with issue

* convert battery+brake

* convert lidar (issue on lidar.wbt)

* convert motor2

* convert gps

* Fix lidar (#3755)

* convert emitter + position sensor

* Revert CoM changes

* fix sickLDMrs proto + convert sick_point_cloud

* change sick point controller

* convert radar

* convert linear motor

* convert connector

* convert lightsensor

* convert sick

* convert gps lat long

* convert speaker

* convert distance sensor + hinge joint + speaker

* convert inertial unit + motor3

* convert motor

* convert range finder

* convert coupled motor

* convert receiver_noise

* convert display

* convert supervisor

* Sample geometries and rendering worlds and protos to ENU/FLU (#3664)

* High resolution IndexedFaceSet world

* polygons

* Textured boxes

* wip

* Improved floating geometries

* Fixed fluid dynamics

* restored default values

* Geometric primitives

* extended solids

* Muscle

* extrusion

* textured shapes

* simplified

* ENU conversion

* enu

* enu

* FLU & ENU

* ENU conversion

* ENU, but not yet FLU

* Teapot in FLU

* Fixed salamander controller

* ENU

* Removed default value for coordinateSystem

* Fixed Viewpoint and re-saved from Webots

* Fix consistency with master

* Update projects/samples/geometries/worlds/textured_shapes.wbt

Co-authored-by: ad-daniel <44834743+ad-daniel@users.noreply.github.com>

* Fixed initial position and behavior of Hinge2 in muscle

Co-authored-by: ad-daniel <44834743+ad-daniel@users.noreply.github.com>

* convert laser_pointer

* display supervisor + convert laser_pointer

* small fix display

* convert gyro

* convert track

* convert propeller

* fix e-puck + convert e-puck.wbt

* fix values sensors e-puckgroundSensors

* convert e-puck world

* convert epuck worlds

* fix viewpoint

* fix youbot

* Update projects/samples/robotbenchmark/pick_and_place/controllers/pick_and_place_benchmark/pick_and_place_benchmark.py

Co-authored-by: Olivier Michel <Olivier.Michel@cyberbotics.com>

* e-puck

* convert curriculum

* fix linear camera

* convert matlab

* fix  linear camera

* Update projects/robots/kuka/youbot/libraries/youbot_control/src/base.c

Co-authored-by: Olivier Michel <Olivier.Michel@cyberbotics.com>

* Update projects/samples/robotbenchmark/pick_and_place/controllers/pick_and_place_benchmark/pick_and_place_benchmark.py

Co-authored-by: Olivier Michel <Olivier.Michel@cyberbotics.com>

* fix proto space + odds + y

* change Group to Transform

* compliance

* ClangFormat compliance

* convert robot window

* fix  epuck flag

* fix pi puck rotation

* convert ball controller

* compliance

* compliance

* cpp check

* Removed useless commented code

* Set rotation in Solid instead of adding a Transform node

* spherical_camera

* FLU: correct inertiaMatrix (#3776)

* bbq and wateringcan

* end of garden

* factory

* balls

* street furniture

* kitchen

* key+gripper

* tiago titanium

* tiago left hand and arm

* test robot urdf tiago

* Update projects/objects/garden/protos/TableWithUmbrella.proto

Co-authored-by: ad-daniel <44834743+ad-daniel@users.noreply.github.com>

Co-authored-by: ad-daniel <44834743+ad-daniel@users.noreply.github.com>

* convert youbot

* convert maze runner

* touch sensors

* convert obstacle avoidance

* FLU: irb4600, surveyor, sojourner (#3750)

* inverse_kinematics.wbt

* surveyor wip

* surveyor

* srv-1.wbt

* sojourner

* inverse kinematics controller

* CoM

* fix CoM Sojourner

* Update projects/robots/kuka/youbot/protos/Youbot.proto

Co-authored-by: Olivier Michel <Olivier.Michel@cyberbotics.com>

* elisa3

* Fix CoM Test (#3791)

* Update projects/samples/devices/worlds/bumper.wbt

Co-authored-by: Benjamin Délèze <benjamin.deleze@epfl.ch>

* Update projects/samples/devices/worlds/pen.wbt

Co-authored-by: Benjamin Délèze <benjamin.deleze@epfl.ch>

* Update projects/samples/devices/worlds/camera_recognition.wbt

Co-authored-by: Benjamin Délèze <benjamin.deleze@epfl.ch>

* Update projects/samples/devices/worlds/camera_auto_focus.wbt

Co-authored-by: Benjamin Délèze <benjamin.deleze@epfl.ch>

* Update projects/samples/devices/worlds/linear_motor.wbt

Co-authored-by: Benjamin Délèze <benjamin.deleze@epfl.ch>

* Update projects/samples/devices/worlds/motor.wbt

Co-authored-by: Benjamin Délèze <benjamin.deleze@epfl.ch>

* Update projects/samples/devices/worlds/connector.wbt

Co-authored-by: Benjamin Délèze <benjamin.deleze@epfl.ch>

* Update projects/samples/devices/worlds/light_sensor.wbt

Co-authored-by: Benjamin Délèze <benjamin.deleze@epfl.ch>

* Update projects/samples/devices/worlds/propeller.wbt

Co-authored-by: Benjamin Délèze <benjamin.deleze@epfl.ch>

* Update projects/samples/devices/worlds/hinge_joint_with_backlash.wbt

Co-authored-by: Benjamin Délèze <benjamin.deleze@epfl.ch>

* Update projects/samples/devices/worlds/track.wbt

Co-authored-by: Benjamin Délèze <benjamin.deleze@epfl.ch>

* Update projects/samples/devices/worlds/inertial_unit.wbt

Co-authored-by: Benjamin Délèze <benjamin.deleze@epfl.ch>

* Update projects/samples/devices/worlds/range_finder.wbt

Co-authored-by: Benjamin Délèze <benjamin.deleze@epfl.ch>

* Update projects/samples/devices/worlds/coupled_motors.wbt

Co-authored-by: Benjamin Délèze <benjamin.deleze@epfl.ch>

* Update projects/samples/devices/worlds/display.wbt

Co-authored-by: Benjamin Délèze <benjamin.deleze@epfl.ch>

* Update projects/samples/devices/worlds/coupled_motors.wbt

Co-authored-by: Benjamin Délèze <benjamin.deleze@epfl.ch>

* Update projects/samples/devices/worlds/motor.wbt

Co-authored-by: Benjamin Délèze <benjamin.deleze@epfl.ch>

* Update projects/samples/devices/worlds/motor.wbt

Co-authored-by: Benjamin Délèze <benjamin.deleze@epfl.ch>

* Update projects/samples/devices/worlds/laser_pointer.wbt

Co-authored-by: Benjamin Délèze <benjamin.deleze@epfl.ch>

* Update projects/samples/devices/worlds/hinge_2_joint_with_backlash.wbt

Co-authored-by: Benjamin Délèze <benjamin.deleze@epfl.ch>

* Update projects/samples/robotbenchmark/maze_runner/worlds/maze_runner.wbt

Co-authored-by: Benjamin Délèze <benjamin.deleze@epfl.ch>

* Update projects/samples/robotbenchmark/maze_runner/worlds/maze_runner.wbt

Co-authored-by: Benjamin Délèze <benjamin.deleze@epfl.ch>

* Update projects/samples/robotbenchmark/maze_runner/worlds/maze_runner.wbt

Co-authored-by: Benjamin Délèze <benjamin.deleze@epfl.ch>

* Update projects/samples/robotbenchmark/maze_runner/worlds/maze_runner.wbt

Co-authored-by: Benjamin Délèze <benjamin.deleze@epfl.ch>

* Update projects/samples/robotbenchmark/maze_runner/worlds/maze_runner.wbt

Co-authored-by: Benjamin Délèze <benjamin.deleze@epfl.ch>

* Update projects/samples/robotbenchmark/maze_runner/worlds/maze_runner.wbt

Co-authored-by: Benjamin Délèze <benjamin.deleze@epfl.ch>

* Update projects/samples/robotbenchmark/maze_runner/worlds/maze_runner.wbt

Co-authored-by: Benjamin Délèze <benjamin.deleze@epfl.ch>

* Update projects/samples/robotbenchmark/maze_runner/worlds/maze_runner.wbt

Co-authored-by: Benjamin Délèze <benjamin.deleze@epfl.ch>

* Update projects/samples/robotbenchmark/maze_runner/worlds/maze_runner.wbt

Co-authored-by: Benjamin Délèze <benjamin.deleze@epfl.ch>

* Update projects/samples/robotbenchmark/maze_runner/worlds/maze_runner.wbt

Co-authored-by: Benjamin Délèze <benjamin.deleze@epfl.ch>

* Update projects/samples/robotbenchmark/maze_runner/worlds/maze_runner.wbt

Co-authored-by: Benjamin Délèze <benjamin.deleze@epfl.ch>

* Update projects/samples/devices/worlds/camera_auto_focus.wbt

Co-authored-by: Benjamin Délèze <benjamin.deleze@epfl.ch>

* Update projects/samples/devices/worlds/hokuyo.wbt

Co-authored-by: Benjamin Délèze <benjamin.deleze@epfl.ch>

* Update projects/samples/devices/worlds/brake.wbt

Co-authored-by: Benjamin Délèze <benjamin.deleze@epfl.ch>

* Update projects/samples/devices/worlds/hokuyo.wbt

Co-authored-by: Benjamin Délèze <benjamin.deleze@epfl.ch>

* Update projects/samples/devices/worlds/hokuyo.wbt

Co-authored-by: Benjamin Délèze <benjamin.deleze@epfl.ch>

* Update projects/samples/robotbenchmark/maze_runner/worlds/maze_runner.wbt

Co-authored-by: Benjamin Délèze <benjamin.deleze@epfl.ch>

* Update projects/samples/devices/worlds/emitter_receiver.wbt

Co-authored-by: Benjamin Délèze <benjamin.deleze@epfl.ch>

* Update projects/samples/devices/worlds/camera.wbt

Co-authored-by: Benjamin Délèze <benjamin.deleze@epfl.ch>

* Update projects/samples/robotbenchmark/maze_runner/worlds/maze_runner.wbt

Co-authored-by: Benjamin Délèze <benjamin.deleze@epfl.ch>

* Update projects/samples/robotbenchmark/maze_runner/worlds/maze_runner.wbt

Co-authored-by: Benjamin Délèze <benjamin.deleze@epfl.ch>

* Update projects/samples/robotbenchmark/maze_runner/worlds/maze_runner.wbt

Co-authored-by: Benjamin Délèze <benjamin.deleze@epfl.ch>

* Update projects/samples/robotbenchmark/maze_runner/worlds/maze_runner.wbt

Co-authored-by: Benjamin Délèze <benjamin.deleze@epfl.ch>

* Update projects/samples/robotbenchmark/maze_runner/worlds/maze_runner.wbt

Co-authored-by: Benjamin Délèze <benjamin.deleze@epfl.ch>

* Update projects/samples/robotbenchmark/maze_runner/worlds/maze_runner.wbt

Co-authored-by: Benjamin Délèze <benjamin.deleze@epfl.ch>

* Update projects/samples/robotbenchmark/maze_runner/worlds/maze_runner.wbt

Co-authored-by: Benjamin Délèze <benjamin.deleze@epfl.ch>

* Update projects/samples/robotbenchmark/maze_runner/worlds/maze_runner.wbt

Co-authored-by: Benjamin Délèze <benjamin.deleze@epfl.ch>

* Update projects/samples/robotbenchmark/obstacle_avoidance/controllers/supervisor/supervisor.py

Co-authored-by: Benjamin Délèze <benjamin.deleze@epfl.ch>

* small fixes

* elisa3.wbt

* clean rotation

* clean rotation

* fix accelerometer leds

* convert led.wbt

* fix compass

* ghostdog

* fix position camera recognition

* FLU: kondo robots (#3733)

* kondo

* khr2 worlds

* khr3

* create

* anaglyph

* create.wbt

* apartement walls

* apartment

* rotate e-puck

* Update projects/robots/kondo/khr-2hv/protos/Khr2hv.proto

Co-authored-by: ad-daniel <44834743+ad-daniel@users.noreply.github.com>

* Update projects/robots/kondo/khr-2hv/protos/Khr2hv.proto

Co-authored-by: ad-daniel <44834743+ad-daniel@users.noreply.github.com>

* Update projects/robots/kondo/khr-2hv/protos/Khr2hv.proto

Co-authored-by: ad-daniel <44834743+ad-daniel@users.noreply.github.com>

* Update projects/robots/kondo/khr-2hv/protos/Khr2hv.proto

Co-authored-by: ad-daniel <44834743+ad-daniel@users.noreply.github.com>

* Update projects/robots/kondo/khr-2hv/protos/Khr2hv.proto

Co-authored-by: ad-daniel <44834743+ad-daniel@users.noreply.github.com>

* Update projects/robots/kondo/khr-2hv/protos/Khr2hv.proto

Co-autho

File: tests/api/controllers/robot_urdf/prob3_reference.urdf (robot description, URDF)
Before this commit: robot P-Rob3, 29 links, 28 joints
Joints:
- joint base_link_cap screw_joint: origin xyz=0.0962 0 0.099 rpy=3.141593 -1.570792 3.141593 -> xyz=0.0962 0 0.099 rpy=0 0 3.141593
- joint link_6_top_button 0_joint: origin xyz=-0.05018 0.043204 0.0089 rpy=0 0 0.9163 -> xyz=-0.05018 0.043204 0.0089 rpy=-1.570796 0 0.9163
- joint link_6_top_button 1_joint: origin xyz=-0.064313 0.015109 0.0089 rpy=0 0 1.309 -> xyz=-0.064313 0.015109 0.0089 rpy=-1.570796 0 1.309
- joint link_6_top_button 2_joint: origin xyz=-0.064201 -0.015644 0.0089 rpy=0 0 1.8 -> xyz=-0.064201 -0.015644 0.0089 rpy=-1.570796 0 1.8
- joint link_6_top_button 3_joint: origin xyz=-0.05053 -0.043194 0.0089 rpy=0 0 2.28 -> xyz=-0.05053 -0.043194 0.0089 rpy=-1.570796 0 2.28
- joint link_6_top_button 4_joint: origin xyz=0.050259 -0.043265 0.0089 rpy=0 0 0.9163 -> xyz=0.050259 -0.043265 0.0089 rpy=-1.570796 0 0.9163
- joint link_6_top_button 5_joint: origin xyz=0.064216 -0.015083 0.0089 rpy=0 0 1.309 -> xyz=0.064216 -0.015083 0.0089 rpy=-1.570796 0 1.309
- joint link_6_top_button 6_joint: origin xyz=0.064201 0.015645 0.0089 rpy=0 0 1.8 -> xyz=0.064201 0.015645 0.0089 rpy=-1.570796 0 1.8
- joint link_6_top_button 7_joint: origin xyz=0.050302 0.042999 0.0089 rpy=0 0 2.28 -> xyz=0.050302 0.042999 0.0089 rpy=-1.570796 0 2.28

Commit message: update urdf test

File: tests/api/controllers/robot_urdf/prob3_reference.urdf (robot description, URDF)
Before this commit: robot P-Rob3, 29 links, 28 joints
Joints:
- joint left finger_left finger sensor 0_joint: origin xyz=0.013 0.02 0.118 rpy=0 0 0 -> xyz=0.013 0.02 0.118 rpy=0.523602 0 0
- joint left finger_left finger sensor 1_joint: origin xyz=-0.013 0.02 0.118 rpy=0 0 3.141593 -> xyz=-0.013 0.02 0.118 rpy=0.523599 0.000001 3.14159
- joint left finger_left finger sensor 2_joint: origin xyz=0 0.021438 0.13449 rpy=-0.000003 -1.125744 -1.570795 -> xyz=0 0.021438 0.13449 rpy=0.523597 -1.125744 -1.570798
- joint left finger_left finger sensor 3_joint: origin xyz=0 0.017324 0.087181 rpy=0.000001 0.261799 1.570802 -> xyz=0 0.017324 0.087181 rpy=0.523601 0.261799 1.570808
- joint right finger_right finger sensor 0_joint: origin xyz=0.013 0.02 0.118 rpy=0 0 0 -> xyz=0.013 0.02 0.118 rpy=0.523599 0 0
- joint right finger_right finger sensor 1_joint: origin xyz=-0.013 0.02 0.118 rpy=0 0 3.141593 -> xyz=-0.013 0.02 0.118 rpy=0.523599 0.000001 3.14159
- joint right finger_right finger sensor 2_joint: origin xyz=0 0.021438 0.13449 rpy=-0.000003 -1.125744 -1.570795 -> xyz=0 0.021438 0.13449 rpy=0.523597 -1.125744 -1.570798
- joint right finger_right finger sensor 3_joint: origin xyz=0 0.017324 0.087181 rpy=0.000001 0.261799 1.570802 -> xyz=0 0.017324 0.087181 rpy=0.523599 0.261799 1.570803
